File: hardware/modules/TrackerOld/TrackerOld.kicad_sch (KiCad schematic)
At the start: 1 part

Commit message: Trackerとりあえず並べました
Parts:
- removed BT101: Battery_Cell, WOBClibrary:cr1220, symbol Device:Battery_Cell
Connections:
- no-connect marks 2 -> 0
Other:
- sheet ESP32 ports: added CANH, CANL; removed CANRX, CANTX, VUSB
- sheet Lipo ports: added none; removed VBUS
