File: hardware/components/GPSPassive/GPSPassive.kicad_sch (KiCad schematic)
At the start: 11 parts, among them U101 NEO-M9N-00B

Commit message: 各コンポーネントの修正をしました．一度プッシュします(多分コンフリクトするので)．
Parts:
- U101: footprint WOBClibrary:SMT_9N-00B_UBL -> WOBCLibrary:ATGM332D-5N31
Connections:
- net GPSANT1: no longer U101.9 (VCC_RF)
- new net VCCRF: U101.9 (VCC_RF)
Changed lines of the file:
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@@
-	)
-	(junction
-		(at 148.59 64.77)
-		(diameter 0)
-		(color 0 0 0 0)
 	)
 	(junction
@@
 	(wire
 		(pts
-			(xy 148.59 74.93) (xy 148.59 64.77)
-		)
-		(stroke
-			(width 0)
-			(type default)
-		)
-	)
-	(wire
-		(pts
 			(xy 114.3 116.84) (xy 114.3 114.3)
 		)
@@
 	(wire
 		(pts
-			(xy 148.59 64.77) (xy 167.64 64.77)
+			(xy 137.795 64.77) (xy 167.64 64.77)
 		)
 		(stroke
@@
 	(wire
 		(pts
-			(xy 137.795 64.77) (xy 148.59 64.77)
-		)
-		(stroke
-			(width 0)
-			(type default)
-		)
-	)
-	(wire
-		(pts
 			(xy 81.915 106.68) (xy 73.66 106.68)
 		)
@@
 		(pts
 			(xy 89.535 139.7) (xy 89.535 134.62)
-		)
-		(stroke
-			(width 0)
-			(type default)
-		)
-	)
-	(wire
-		(pts
-			(xy 135.89 74.93) (xy 148.59 74.93)
 		)
 		(stroke
@@
 		(property "Intersheetrefs" "${INTERSHEET_REFS}"
 			(at 131.9976 127 0)
-			(effects
-				(font
-					(size 1.27 1.27)
-				)
-				(justify right)
-				(hide yes)
-			)
-		)
-	)
-	(global_label "VCCRF"
-		(shape input)
-		(at 135.89 74.93 180)
-		(fields_autoplaced yes)
-		(effects
-			(font
-				(size 1.27 1.27)
-			)
-			(justify right)
-		)
-		(property "Intersheetrefs" "${INTERSHEET_REFS}"
-			(at 126.9176 74.93 0)
 			(effects
 				(font
@@
 			)
 		)
-		(property "Footprint" "WOBClibrary:SMT_9N-00B_UBL"
+		(property "Footprint" "WOBCLibrary:ATGM332D-5N31"
 			(at 143.51 106.68 0)
 			(effects
@@
 		)
 	)
+	(sheet_instances
+		(path "/"
+			(page "1")
+		)
+	)
