File: hardware/components/LCD/LCD.kicad_sch (KiCad schematic)
At the start: 50 parts, among them J101 Conn_01x04_MountingPin, SW101 sw1, SW102 sw1, SW103 sw1, SW104 sw1, SW105 sw1, SW106 sw1, SW107 sw1

Commit message: コメントもらった分修正加えました。LiPoのLCSC、RP2040CoreのUSB-C、LCDのプルアップ抵抗です。 USB-Cはフットプリント作ったやつで不安なので、確認してもらいたいです。
Parts:
- R101, R103, R104, R105, R106, R107, R108, R109, R110, R111, R112: value 3K3 -> 47k; LCSC C25890 -> C25792
- R113, R114, R115, R116, R117, R118, R119, R120, R121, R122, R123, R124, R125, R126: LCSC C25890 -> C11702
Changed lines of the file:
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@@
 			)
 		)
-		(property "LCSC" "C25890 "
+		(property "LCSC" "C11702"
 			(at 134 150 0)
 			(effects
@@
 			)
 		)
-		(property "LCSC" "C25890 "
+		(property "LCSC" "C11702"
 			(at 84 180 0)
 			(effects
@@
 			)
 		)
-		(property "LCSC" "C25890 "
+		(property "LCSC" "C11702"
 			(at 40 160 0)
 			(effects
@@
 			)
 		)
-		(property "LCSC" "C25890 "
+		(property "LCSC" "C11702"
 			(at 84 170 0)
 			(effects
@@
 			)
 		)
-		(property "Value" "3K3"
+		(property "Value" "47k"
 			(at 153.2149 31.5985 90)
 			(effects
@@
 			)
 		)
-		(property "LCSC" "C25890 "
+		(property "LCSC" "C25792"
 			(at 155.7549 34.1385 0)
 			(effects
@@
 			)
 		)
-		(property "LCSC" "C25890 "
+		(property "LCSC" "C11702"
 			(at 40 180 0)
 			(effects
@@
 			)
 		)
-		(property "LCSC" "C25890 "
+		(property "LCSC" "C11702"
 			(at 85 110 0)
 			(effects
@@
 			)
 		)
-		(property "LCSC" "C25890 "
+		(property "LCSC" "C11702"
 			(at 40 120 0)
 			(effects
@@
 			)
 		)
-		(property "Value" "3K3"
+		(property "Value" "47k"
 			(at 55.4169 68.2078 90)
 			(effects
@@
 			)
 		)
-		(property "LCSC" "C25890 "
+		(property "LCSC" "C25792"
 			(at 52.8769 65.6678 0)
 			(effects
@@
 			)
 		)
-		(property "LCSC" "C25890 "
+		(property "LCSC" "C11702"
 			(at 84 150 0)
 			(effects
@@
 			)
 		)
-		(property "Value" "3K3"
+		(property "Value" "47k"
 			(at 218.6273 40.835 90)
 			(effects
@@
 			)
 		)
-		(property "LCSC" "C25890 "
+		(property "LCSC" "C25792"
 			(at 221.1673 43.375 0)
 			(effects
@@
 			)
 		)
-		(property "LCSC" "C25890 "
+		(property "LCSC" "C11702"
 			(at 40 130 0)
 			(effects
@@
 			)
 		)
-		(property "Value" "3K3"
+		(property "Value" "47k"
 			(at 148.1349 31.5985 90)
 			(effects
@@
 			)
 		)
-		(property "LCSC" "C25890 "
+		(property "LCSC" "C25792"
 			(at 150.6749 34.1385 0)
 			(effects
@@
 			)
 		)
-		(property "Value" "3K3"
+		(property "Value" "47k"
 			(at 159.0532 31.9171 90)
 			(effects
@@
 			)
 		)
-		(property "LCSC" "C25890 "
+		(property "LCSC" "C25792"
 			(at 161.5932 34.4571 0)
 			(effects
@@
 			)
 		)
-		(property "LCSC" "C25890 "
+		(property "LCSC" "C11702"
 			(at 40 150 0)
 			(effects
@@
 			)
 		)
-		(property "LCSC" "C25890 "
+		(property "LCSC" "C11702"
 			(at 40 170 0)
 			(effects
@@
 			)
 		)
-		(property "Value" "3K3"
+		(property "Value" "47k"
 			(at 164.9231 32.0505 90)
 			(effects
@@
 			)
 		)
-		(property "LCSC" "C25890 "
+		(property "LCSC" "C25792"
 			(at 167.4631 34.5905 0)
 			(effects
@@
 			)
 		)
-		(property "LCSC" "C25890 "
+		(property "LCSC" "C11702"
 			(at 40 110 0)
 			(effects
@@
 			)
 		)
-		(property "Value" "3K3"
+		(property "Value" "47k"
 			(at 213.5473 40.835 90)
 			(effects
@@
 			)
 		)
-		(property "LCSC" "C25890 "
+		(property "LCSC" "C25792"
 			(at 216.0873 43.375 0)
 			(effects
@@
 			)
 		)
-		(property "Value" "3K3"
+		(property "Value" "47k"
 			(at 241.4417 41.0277 90)
 			(effects
@@
 			)
 		)
-		(property "LCSC" "C25890 "
+		(property "LCSC" "C25792"
 			(at 243.9817 43.5677 0)
 			(effects
@@
 			)
 		)
-		(property "Value" "3K3"
+		(property "Value" "47k"
 			(at 224.4656 41.1536 90)
 			(effects
@@
 			)
 		)
-		(property "LCSC" "C25890 "
+		(property "LCSC" "C25792"
 			(at 227.0056 43.6936 0)
 			(effects
@@
 			)
 		)
-		(property "LCSC" "C25890 "
+		(property "LCSC" "C11702"
 			(at 84 160 0)
 			(effects
@@
 			)
 		)
-		(property "Value" "3K3"
+		(property "Value" "47k"
 			(at 235.9693 41.0277 90)
 			(effects
@@
 			)
 		)
-		(property "LCSC" "C25890 "
+		(property "LCSC" "C25792"
 			(at 238.5093 43.5677 0)
 			(effects
@@
 			)
 		)
-		(property "LCSC" "C25890 "
+		(property "LCSC" "C11702"
 			(at 85 120 0)
 			(effects
@@
 			)
 		)
-		(property "Value" "3K3"
+		(property "Value" "47k"
 			(at 230.3355 41.287 90)
 			(effects
@@
 			)
 		)
-		(property "LCSC" "C25890 "
+		(property "LCSC" "C25792"
 			(at 232.8755 43.827 0)
 			(effects

Commit message: USB-Cのフットプリントの変更・GSモジュールの回路図配線完了しました。 Coreの方はUSB-Cのフットプリント修正してますので、こちらを使ってもらえればと思います。
Parts:
- removed R117, R118, R119, R120, R121, R122, R123, R124, R125, R126: 1k, Capacitor_SMD:C_0402_1005Metric, symbol Device:R_US
Connections:
- net GND: no longer D101.1 (K), D102.1 (K), D103.1 (K), D104.1 (K), D105.1 (K), D106.1 (K), D107.1 (K), D108.1 (K), D109.1 (K), D110.1 (K), D111.1 (K), D112.1 (K), D113.1 (K), D114.1 (K)
- net at D112.2 (A): now also D103.2 (A), D106.2 (A), D110.2 (A), R114.2
- net at D111.2 (A): now also D107.2 (A), R113.2
- net at D105.2 (A): now also D102.2 (A), D109.2 (A), D114.2 (A), R115.2
- net at D104.2 (A), R116.2: now also D101.2 (A), D108.2 (A), D113.2 (A)
- net Power_Charge renamed ind_column2
- net Power_ON renamed ind_column4
- net Power_Shortage renamed ind_column3
- net RS1_Receive renamed ind_column1
- new net ind_row1: D101.1 (K), D102.1 (K), D103.1 (K)
- new net ind_row2: D112.1 (K), D113.1 (K), D114.1 (K)
- new net ind_row3: D104.1 (K), D105.1 (K), D106.1 (K), D107.1 (K)
- new net ind_row4: D108.1 (K), D109.1 (K), D110.1 (K), D111.1 (K)
- no-connect marks 41 -> 35
Other:
- moved on the sheet: D101, D102, D103, D104, D105, D106, D107, D108, D109, D110, D111, D112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

Commit message: 各コンポーネントの修正をしました．一度プッシュします(多分コンフリクトするので)．
Parts:
- renumbered D112 to D10, D106 to D11, D103 to D12, D109 to D13, D114 to D14, D105 to D15, D102 to D16, D108 to D17, D113 to D18, D104 to D19, D101 to D20, D111 to D7, D107 to D8, D110 to D9, J101 to J4, R101 to R14, R102 to R15, R113 to R16, R114 to R17, R115 to R18, R116 to R19, R109 to R20, R110 to R21, R111 to R22, R112 to R23, R103 to R24, R104 to R25, R105 to R26, R106 to R27, R107 to R28, R108 to R29, SW101 to SW10, SW103 to SW3, SW108 to SW4, SW106 to SW5, SW107 to SW6, SW104 to SW7, SW105 to SW8, SW102 to SW9, lcd101 to lcd1
