File: hardware/components/Logger/Logger.kicad_pcb (KiCad board)
At the start: 2 copper layers, 5 parts, among them U1 PCF8563T, Y1 Crystal

Commit message: 各コンポーネントの修正をしました．一度プッシュします(多分コンフリクトするので)．
Parts:
- renumbered C1 to C101, C2 to C102, MICRO_SD1 to MICRO_SD101, U1 to U101, Y1 to Y101
Changed lines of the file:
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@@
 	(net 3 "+BATT")
 	(net 4 "/SD_MOSI")
-	(net 5 "unconnected-(MICRO_SD1-DAT1-Pad8)")
+	(net 5 "unconnected-(MICRO_SD101-DAT1-Pad8)")
 	(net 6 "/SD_DET")
-	(net 7 "unconnected-(MICRO_SD1-DAT2-Pad1)")
+	(net 7 "unconnected-(MICRO_SD101-DAT2-Pad1)")
 	(net 8 "/SD_CLK")
 	(net 9 "/SD_MISO")
@@
 	(net 11 "/I2C_SDA")
 	(net 12 "/I2C_SCL")
-	(net 13 "unconnected-(U1-~{INT}-Pad3)")
-	(net 14 "Net-(U1-OSCI)")
-	(net 15 "Net-(U1-OSCO)")
-	(net 16 "unconnected-(U1-CLKO-Pad7)")
+	(net 13 "unconnected-(U101-~{INT}-Pad3)")
+	(net 14 "Net-(U101-OSCI)")
+	(net 15 "Net-(U101-OSCO)")
+	(net 16 "unconnected-(U101-CLKO-Pad7)")
 	(footprint "Package_SO:SOIC-8_3.9x4.9mm_P1.27mm"
 		(layer "F.Cu")
@@
 		(descr "SOIC, 8 Pin (JEDEC MS-012AA, https://www.analog.com/media/en/package-pcb-resources/package/pkg_pdf/soic_narrow-r/r_8.pdf), generated with kicad-footprint-generator ipc_gullwing_generator.py")
 		(tags "SOIC SO")
-		(property "Reference" "U1"
+		(property "Reference" "U101"
 			(at 0 -3.4 0)
 			(layer "F.SilkS")
@@
 				(font
 					(size 1.27 1.27)
+				)
+			)
+		)
+		(property "LCSC" "C7440"
+			(at 0 0 0)
+			(unlocked yes)
+			(layer "F.Fab")
+			(hide yes)
+			(effects
+				(font
+					(size 1 1)
+					(thickness 0.15)
 				)
 			)
@@
 			(layers "F.Cu" "F.Paste" "F.Mask")
 			(roundrect_rratio 0.25)
-			(net 14 "Net-(U1-OSCI)")
+			(net 14 "Net-(U101-OSCI)")
 			(pinfunction "OSCI")
 			(pintype "input")
@@
 			(layers "F.Cu" "F.Paste" "F.Mask")
 			(roundrect_rratio 0.25)
-			(net 15 "Net-(U1-OSCO)")
+			(net 15 "Net-(U101-OSCO)")
 			(pinfunction "OSCO")
 			(pintype "output")
@@
 			(layers "F.Cu" "F.Paste" "F.Mask")
 			(roundrect_rratio 0.25)
-			(net 13 "unconnected-(U1-~{INT}-Pad3)")
+			(net 13 "unconnected-(U101-~{INT}-Pad3)")
 			(pinfunction "~{INT}")
 			(pintype "output+no_connect")
@@
 			(layers "F.Cu" "F.Paste" "F.Mask")
 			(roundrect_rratio 0.25)
-			(net 16 "unconnected-(U1-CLKO-Pad7)")
+			(net 16 "unconnected-(U101-CLKO-Pad7)")
 			(pinfunction "CLKO")
 			(pintype "output+no_connect")
@@
 		(at 154.895 97.645)
 		(descr "<b>TF-01A-6</b><br>")
-		(property "Reference" "MICRO_SD1"
+		(property "Reference" "MICRO_SD101"
 			(at -2.54 -5.024 0)
 			(layer "F.SilkS")
@@
 		)
 		(property "Check_prices" "https://www.snapeda.com/parts/TF-01A/HRO+Electronics+Co.%252C+Ltd./view-part/?ref=eda"
+			(at 0 0 0)
+			(unlocked yes)
+			(layer "F.Fab")
+			(hide yes)
+			(effects
+				(font
+					(size 1 1)
+					(thickness 0.15)
+				)
+			)
+		)
+		(property "LCSC" "C5155563"
 			(at 0 0 0)
 			(unlocked yes)
@@
 			(size 1.3 0.7)
 			(layers "F.Cu" "F.Paste" "F.Mask")
-			(net 7 "unconnected-(MICRO_SD1-DAT2-Pad1)")
+			(net 7 "unconnected-(MICRO_SD101-DAT2-Pad1)")
 			(pinfunction "DAT2")
 			(pintype "bidirectional+no_connect")
@@
 			(size 1.3 0.7)
 			(layers "F.Cu" "F.Paste" "F.Mask")
-			(net 5 "unconnected-(MICRO_SD1-DAT1-Pad8)")
+			(net 5 "unconnected-(MICRO_SD101-DAT1-Pad8)")
 			(pinfunction "DAT1")
 			(pintype "bidirectional+no_connect")
@@
 		(descr "Capacitor SMD 0402 (1005 Metric), square (rectangular) end terminal, IPC_7351 nominal, (Body size source: IPC-SM-782 page 76, https://www.pcb-3d.com/wordpress/wp-content/uploads/ipc-sm-782a_amendment_1_and_2.pdf), generated with kicad-footprint-generator")
 		(tags "capacitor")
-		(property "Reference" "C2"
+		(property "Reference" "C102"
 			(at 0 -1.16 0)
 			(layer "F.SilkS")
@@
 				(font
 					(size 1.27 1.27)
+				)
+			)
+		)
+		(property "LCSC" "C1525"
+			(at 0 0 0)
+			(unlocked yes)
+			(layer "F.Fab")
+			(hide yes)
+			(effects
+				(font
+					(size 1 1)
+					(thickness 0.15)
 				)
 			)
@@
 		(descr "SMD Crystal FC-135 https://support.epson.biz/td/api/doc_check.php?dl=brief_FC-135R_en.pdf")
 		(tags "SMD SMT Crystal")
-		(property "Reference" "Y1"
+		(property "Reference" "Y101"
 			(at 0 -2 0)
 			(layer "F.SilkS")
@@
 				(font
 					(size 1.27 1.27)
+				)
+			)
+		)
+		(property "LCSC" "C9002"
+			(at 0 0 0)
+			(unlocked yes)
+			(layer "F.Fab")
+			(hide yes)
+			(effects
+				(font
+					(size 1 1)
+					(thickness 0.15)
 				)
 			)
@@
 			(size 1 1.8)
 			(layers "F.Cu" "F.Paste" "F.Mask")
-			(net 14 "Net-(U1-OSCI)")
+			(net 14 "Net-(U101-OSCI)")
 			(pinfunction "1")
 			(pintype "passive")
@@
 			(size 1 1.8)
 			(layers "F.Cu" "F.Paste" "F.Mask")
-			(net 15 "Net-(U1-OSCO)")
+			(net 15 "Net-(U101-OSCO)")
 			(pinfunction "2")
 			(pintype "passive")
@@
 		(descr "Capacitor SMD 0402 (1005 Metric), square (rectangular) end terminal, IPC_7351 nominal, (Body size source: IPC-SM-782 page 76, https://www.pcb-3d.com/wordpress/wp-content/uploads/ipc-sm-782a_amendment_1_and_2.pdf), generated with kicad-footprint-generator")
 		(tags "capacitor")
-		(property "Reference" "C1"
+		(property "Reference" "C101"
 			(at 0 -1.16 0)
 			(layer "F.SilkS")
@@
 				)
 			)
+		)
+		(property "LCSC" "C96446"
+			(at 0 0 0)
+			(unlocked yes)
+			(layer "F.Fab")
+			(hide yes)
+			(effects
+				(font
+					(size 1 1)
+					(thickness 0.15)
+				)
+			)
