File: hardware/modules/Controller/RP2040.kicad_sch (KiCad schematic)
At the start: 41 parts, among them J1 DEBUG, SW1 RESET, SW2 BOOT0, U1 SN65HVD230, U2 W25Q128JVS, U3 RP2040, Y1 Crystal_GND24

Commit message: GSモジュール一式完成です．最終確認をお願いします．週末に発注しようと思います．
Parts:
- D1, D5, D6: footprint LED_SMD:LED_0603_1608Metric -> LED_SMD:LED_0805_2012Metric
- SW1: LCSC C2296 -> (none)
Changed lines of the file:
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@@
 			)
 		)
-		(property "Footprint" "LED_SMD:LED_0603_1608Metric"
+		(property "Footprint" "LED_SMD:LED_0805_2012Metric"
 			(at 255.6513 138.5981 0)
 			(effects
@@
 			)
 		)
-		(property "Footprint" "LED_SMD:LED_0603_1608Metric"
+		(property "Footprint" "LED_SMD:LED_0805_2012Metric"
 			(at 58.1663 111.9281 0)
 			(effects
@@
 			)
 		)
-		(property "LCSC" "C2296"
+		(property "LCSC" ""
 			(at 58.1663 123.3581 0)
 			(effects
@@
 			)
 		)
-		(property "Footprint" "LED_SMD:LED_0603_1608Metric"
+		(property "Footprint" "LED_SMD:LED_0805_2012Metric"
 			(at 244.8563 138.5981 0)
 			(effects

Commit message: 部品の割り当てやGPSモジュールのフットプリント修正などです。
Parts:
- C3, C4: LCSC C346183 -> C1555
- SW1: value RESET -> RESET_sw
- SW2: LCSC C720477 -> (none)
Changed lines of the file:
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@@
 			)
 		)
-		(property "LCSC" "C720477"
+		(property "LCSC" ""
 			(at 136.2713 107.4831 0)
 			(effects
@@
 			)
 		)
-		(property "LCSC" " C346183"
+		(property "LCSC" "C1555"
 			(at 154.0513 118.2781 0)
 			(effects
@@
 			)
 		)
-		(property "LCSC" " C346183"
+		(property "LCSC" "C1555"
 			(at 154.0513 108.1181 0)
 			(effects
@@
 			)
 		)
-		(property "Value" "RESET"
+		(property "Value" "RESET_sw"
 			(at 60.7063 127.1681 0)
 			(effects

Commit message: 各コンポーネントの修正をしました．一度プッシュします(多分コンフリクトするので)．
Parts:
- C103: renamed from C1; LCSC C1525 -> C1525
- C104: renamed from C2; LCSC C1525 -> C1525
- C107: renamed from C5; LCSC C1525 -> C1525
- C108: renamed from C6; LCSC C1525 -> C1525
- C109: renamed from C7; LCSC C52923 -> C52923
- C110: renamed from C8; LCSC C1525 -> C1525
- C111: renamed from C9; LCSC C52923 -> C52923
- C112: renamed from C10; LCSC C1525 -> C1525
- C113: renamed from C11; LCSC C1525 -> C1525
- C114: renamed from C12; LCSC C1525 -> C1525
- C115: renamed from C13; LCSC C1525 -> C1525
- C116: renamed from C14; LCSC C1525 -> C1525
- C117: renamed from C15; LCSC C1525 -> C1525
- D106: renamed from D6; LCSC C84256 -> C84256
- R102: renamed from R2; LCSC C11702 -> C11702
- R103: renamed from R3; LCSC C25768 -> C25768
- R104: renamed from R4; LCSC C25768 -> C25768
- R105: renamed from R5; LCSC C11702 -> C11702
- R106: renamed from R6; LCSC C25092 -> C25092
- R107: renamed from R7; LCSC C25092 -> C25092
- R108: renamed from R8; LCSC C11702 -> C11702
- R110: renamed from R10; LCSC C11702 -> C11702
- R112: renamed from R12; LCSC C11702 -> C11702
- U104: renamed from U3; LCSC C2040 -> C2040
- Y101: renamed from Y1; LCSC C9002 -> C9002
- renumbered C3 to C105, C4 to C106, D1 to D101, D2 to D102, D3 to D103, D4 to D104, D5 to D105, J1 to J101, R1 to R101, R9 to R109, R11 to R111, SW1 to SW101, SW2 to SW102, U1 to U102, U2 to U103, USB1 to USB101
