File: hardware/modules/GS/ModuleIFSimple2.kicad_sch (KiCad schematic)
At the start: 4 parts, among them J1 Jumper, J2 Conn_01x04_MountingPin

Commit message: 各コンポーネントの修正をしました．一度プッシュします(多分コンフリクトするので)．
Parts:
- renumbered C6 to C7, R12 to R10
Changed lines of the file:
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@@
 		(dnp no)
 		(fields_autoplaced yes)
-		(property "Reference" "#PWR033"
+		(property "Reference" "#PWR031"
 			(at 187.325 82.55 0)
 			(effects
@@
 			(project "GS"
 				(path "/920f9ee9-d8de-4f24-ad72-1c45434a67fe/b6596e6a-331e-4110-9845-3f13c73105a2"
-					(reference "#PWR033")
+					(reference "#PWR031")
 					(unit 1)
 				)
@@
 		(on_board yes)
 		(dnp no)
-		(property "Reference" "R12"
+		(property "Reference" "R10"
 			(at 175.26 52.705 0)
 			(effects
@@
 			(project "GS"
 				(path "/920f9ee9-d8de-4f24-ad72-1c45434a67fe/b6596e6a-331e-4110-9845-3f13c73105a2"
-					(reference "R12")
+					(reference "R10")
 					(unit 1)
 				)
@@
 		(dnp no)
 		(fields_autoplaced yes)
-		(property "Reference" "#PWR032"
+		(property "Reference" "#PWR030"
 			(at 180.975 82.55 0)
 			(effects
@@
 			(project "GS"
 				(path "/920f9ee9-d8de-4f24-ad72-1c45434a67fe/b6596e6a-331e-4110-9845-3f13c73105a2"
-					(reference "#PWR032")
+					(reference "#PWR030")
 					(unit 1)
 				)
@@
 		(on_board yes)
 		(dnp no)
-		(property "Reference" "C6"
+		(property "Reference" "C7"
 			(at 153.67 75.565 0)
 			(effects
@@
 			(project "GS"
 				(path "/920f9ee9-d8de-4f24-ad72-1c45434a67fe/b6596e6a-331e-4110-9845-3f13c73105a2"
-					(reference "C6")
+					(reference "C7")
 					(unit 1)
 				)
@@
 		(dnp no)
 		(fields_autoplaced yes)
-		(property "Reference" "#PWR031"
+		(property "Reference" "#PWR029"
 			(at 154.94 83.82 0)
 			(effects
@@
 			(project "GS"
 				(path "/920f9ee9-d8de-4f24-ad72-1c45434a67fe/b6596e6a-331e-4110-9845-3f13c73105a2"
-					(reference "#PWR031")
-					(unit 1)
-				)
+					(reference "#PWR029")
+					(unit 1)
+				)
