File: hardware/components/RP2040Core/RP2040Core.kicad_sch (KiCad schematic)
At the start: 41 parts, among them J1 DEBUG, SW1 BOOT0, SW1 RESET, U2 W25Q128JVS, U3 RP2040, U3 SN65HVD230, Y1 Crystal_GND24

Commit message: マージしたので，これでうまくいってほしいです．
Parts:
- C4: LCSC (none) -> C346183
- C4, C6: LCSC (none) -> C1525
- C5: LCSC (none) -> C52923
- D4, SW1: LCSC (none) -> C2296
- D5: LCSC (none) -> C84256
- D6: LCSC (none) -> C2297
- R1: LCSC (none) -> C25092
- R1, R2: LCSC (none) -> C25768
- R3, R5, R7: LCSC (none) -> C25744
- R3, R4, R5, R6: LCSC (none) -> C11702
- SW1: LCSC (none) -> C720477
- U102: renamed from U2; LCSC (none) -> C97521
- U103: renamed from U3; LCSC (none) -> C2040
- U3: now not fitted
- USB1: LCSC (none) -> C2856766
- Y101: renamed from Y1; LCSC (none) -> C9002
- renumbered J1 to J101

Commit message: ESDダイオードの変更などです。GSはまだ作りかけなので参考にしないでください
Parts:
- removed C4: 100nF, Capacitor_SMD:C_0402_1005Metric, symbol Device:C_Small
- removed D1, D2, D3: 5V, Diode_SMD:D_SOD-923, symbol Diode:ESD9B5.0ST5G
- removed D4: RESET, LED_SMD:LED_0603_1608Metric, symbol Device:LED
- removed R1, R2: 22k, Resistor_SMD:R_0402_1005Metric, symbol Device:R
- removed R3: 1k, Resistor_SMD:R_0402_1005Metric, symbol Device:R
- removed R5, R7: 10k, Resistor_SMD:R_0402_1005Metric, symbol Device:R
- removed SW1: RESET, WOBCLibrary:TVAF06-A020B-R, symbol Switch:SW_Push
- removed U3: SN65HVD230, Package_SO:SOIC-8_3.9x4.9mm_P1.27mm, symbol Interface_CAN_LIN:SN65HVD230
- removed USB1: USB_C_Receptacle_USB2.0, Connector_USB:USB_C_Receptacle_XKB_U262-16XN-4BVC11, symbol Connector:USB_C_Receptacle_USB2.0
- added C105: 100nF, Capacitor_SMD:C_0402_1005Metric, symbol Device:C_Small
- added D107: RESET, LED_SMD:LED_0603_1608Metric, symbol Device:LED
- added D108, D109, D110: 5V, Diode_SMD:D_SOD-882, symbol Diode:ESD9B5.0ST5G
- added R113: 1k, Resistor_SMD:R_0402_1005Metric, symbol Device:R
- added R114, R115: 22k, Resistor_SMD:R_0402_1005Metric, symbol Device:R
- added R120, R122: 10k, Resistor_SMD:R_0402_1005Metric, symbol Device:R
- added SW103: RESET, WOBCLibrary:TVAF06-A020B-R, symbol Switch:SW_Push
- added U104: SN65HVD230, Package_SO:SOIC-8_3.9x4.9mm_P1.27mm, symbol Interface_CAN_LIN:SN65HVD230
- added USB102: USB_C_Receptacle_USB2.0, Connector_USB:USB_C_Receptacle_XKB_U262-16XN-4BVC11, symbol Connector:USB_C_Receptacle_USB2.0
- renumbered C4 to C106, C4 to C107, C4 to C108, C6 to C109, C6 to C110, C5 to C111, C6 to C112, C5 to C113, C6 to C114, C6 to C115, C6 to C116, C6 to C117, C6 to C118, C6 to C119, D6 to D111, D5 to D112, J101 to J103, R3 to R112, R5 to R116, R1 to R117, R1 to R118, R5 to R119, R6 to R121, R4 to R123, SW1 to SW104, U102 to U105, U103 to U106
Connections:
- net CANH: now also U104.7 (CANH)
- net CANL: now also U104.6 (CANL)
- net CAN_RX: now also U104.4 (R)
- net CAN_TX: now also U104.1 (D)
- net GND: now also C105.1, D108.1 (A1), D109.1 (A1), D110.1 (A1), R114.2, R115.2, SW103.2, U104.2 (GND), U104.8 (Rs), USB102.A1 (GND), USB102.A12 (GND), USB102.B1 (GND), USB102.B12 (GND), USB102.S1 (SHIELD)
- net I2C_SCL: now also R122.2
- net I2C_SDA: now also R120.2
- net RESET: now also D107.1 (K), SW103.1
- net USB_D+: now also D109.2 (A2), USB102.A6 (D+), USB102.B6 (D+)
- net USB_D-: now also D110.2 (A2), USB102.A7 (D-), USB102.B7 (D-)
- net VBUS: now also D108.2 (A2), USB102.A4 (VBUS), USB102.A9 (VBUS), USB102.B4 (VBUS), USB102.B9 (VBUS)
- net VDD: now also C105.2, R113.1, R120.1, R122.1, U104.3 (VCC)
- new net: R115.1, USB102.B5 (CC2)
- new net: D107.2 (A), R113.2
- new net: R114.1, USB102.A5 (CC1)

Commit message: コメントもらった分修正加えました。LiPoのLCSC、RP2040CoreのUSB-C、LCDのプルアップ抵抗です。 USB-Cはフットプリント作ったやつで不安なので、確認してもらいたいです。
Parts:
- USB102: footprint Connector_USB:USB_C_Receptacle_XKB_U262-16XN-4BVC11 -> WOBCLibrary:USB_C_TYPEC-301S-ACP16X7
Changed lines of the file:
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@@
 			)
 		)
-		(property "Footprint" "Connector_USB:USB_C_Receptacle_XKB_U262-16XN-4BVC11"
+		(property "Footprint" "WOBCLibrary:USB_C_TYPEC-301S-ACP16X7"
 			(at 32.385 41.91 0)
 			(effects
@@
 		)
 	)
+	(sheet_instances
+		(path "/"
+			(page "1")
+		)
+	)

Commit message: 各コンポーネントの修正をしました．一度プッシュします(多分コンフリクトするので)．
Parts:
- C105, C106, C109, C110, C112, C114, C115, C116, C117, C118, C119: LCSC C1525 -> C1525
- C107, C108: LCSC C346183 -> C1555
- C111, C113: LCSC C52923 -> C52923
- D107, D111: footprint LED_SMD:LED_0603_1608Metric -> LED_SMD:LED_0805_2012Metric
- D112: footprint LED_SMD:LED_0603_1608Metric -> LED_SMD:LED_0805_2012Metric; LCSC C84256 -> C84256
- R113, R116, R119, R121, R123: LCSC C11702 -> C11702
- R114, R115: LCSC C25768 -> C25768
- R117, R118: LCSC C25092 -> C25092
- SW103: value RESET -> RESET_sw; LCSC C2296 -> (none)
- SW104: LCSC C720477 -> (none)
- U106: LCSC C2040 -> C2040
- Y101: LCSC C9002 -> C9002

Commit message: Mission基板のオーダーファイルの作成・コンポーネント修正（LiPoバックアップ切り替え、GNSS書き込み、usbプルダウン抵抗）
Parts:
- R114, R115: value 22k -> 5.1k; LCSC C25768 -> C25905
