File: hardware/modules/MissionOrderFile/MissionOrderFile/GS/ModuleIFSimple4.kicad_sch (KiCad schematic)
At the start: 4 parts, among them J101 Jumper, J102 Conn_01x04_MountingPin

Commit message: GS修正＋発注ファイルにGSのデータを反映
Parts:
- removed C107: 100nF, Capacitor_SMD:C_0402_1005Metric, symbol Device:C
- removed J101: Jumper, Connector_PinHeader_1.27mm:PinHeader_1x02_P1.27mm_Vertical, symbol Connector:Conn_01x02_Pin
- removed J102: Conn_01x04_MountingPin, WOBCLibrary:Grove_4P_L_SMD, symbol Connector_Generic_MountingPin:Conn_01x04_MountingPin
- removed R110: 120, Resistor_SMD:R_0402_1005Metric, symbol Device:R
- added C108: 100nF, Capacitor_SMD:C_0402_1005Metric, symbol Device:C
- added J103: Jumper, Connector_PinHeader_1.27mm:PinHeader_1x02_P1.27mm_Vertical, symbol Connector:Conn_01x02_Pin
- added J104: Conn_01x04_MountingPin, WOBCLibrary:Grove_4P_L_SMD, symbol Connector_Generic_MountingPin:Conn_01x04_MountingPin
- added R111: 120, Resistor_SMD:R_0402_1005Metric, symbol Device:R
Connections:
- net CANH: now also J104.1 (Pin_1), R111.2
- net CANL: now also J103.2 (Pin_2), J104.2 (Pin_2)
- net GND: now also C108.1, J104.4 (Pin_4), J104.MP (MountPin)
- net VIO: now also C108.2, J104.3 (Pin_3)
- new net: J103.1 (Pin_1), R111.1
