File: hardware/components/TankPressure/TankPressure.kicad_sch (KiCad schematic)
At the start: 19 parts, among them J101 Conn_01x03, U101 TPS63070RNMR

Commit message: RCS関連コンポーネント修正
Parts:
- L101: value L -> 1.5uH
- R107: value 10k -> 1k; LCSC C25744 -> C11702
Connections:
- net GND: no longer R107.1
- net TankPressure: no longer J101.2 (Pin_2)
- new net: J101.2 (Pin_2), R107.1
Changed lines of the file:
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@@
-	)
-	(junction
-		(at 210.693 92.71)
-		(diameter 0)
-		(color 0 0 0 0)
 	)
 	(junction
@@
 	)
 	(junction
-		(at 201.549 92.71)
-		(diameter 0)
-		(color 0 0 0 0)
-	)
-	(junction
 		(at 91.059 75.946)
 		(diameter 0)
@@
 	(wire
 		(pts
-			(xy 210.693 78.486) (xy 211.455 78.486)
+			(xy 210.566 78.486) (xy 211.455 78.486)
 		)
 		(stroke
@@
 	(wire
 		(pts
-			(xy 210.693 92.71) (xy 210.439 92.71)
-		)
-		(stroke
-			(width 0)
-			(type default)
-		)
-	)
-	(wire
-		(pts
 			(xy 120.269 65.786) (xy 108.204 65.786)
 		)
@@
 	(wire
 		(pts
+			(xy 219.964 92.71) (xy 221.234 92.71)
+		)
+		(stroke
+			(width 0)
+			(type default)
+		)
+	)
+	(wire
+		(pts
 			(xy 100.584 98.171) (xy 100.584 104.521)
 		)
@@
 	(wire
 		(pts
-			(xy 201.549 92.71) (xy 202.819 92.71)
-		)
-		(stroke
-			(width 0)
-			(type default)
-		)
-	)
-	(wire
-		(pts
 			(xy 153.924 88.646) (xy 153.924 75.946)
 		)
@@
 	(wire
 		(pts
+			(xy 210.566 92.71) (xy 212.344 92.71)
+		)
+		(stroke
+			(width 0)
+			(type default)
+		)
+	)
+	(wire
+		(pts
 			(xy 188.595 75.946) (xy 197.739 75.946)
 		)
@@
 	(wire
 		(pts
-			(xy 210.693 92.71) (xy 212.725 92.71)
-		)
-		(stroke
-			(width 0)
-			(type default)
-		)
-	)
-	(wire
-		(pts
-			(xy 210.693 78.486) (xy 210.693 92.71)
+			(xy 210.566 78.486) (xy 210.566 92.71)
 		)
 		(stroke
@@
 	(hierarchical_label "TankPressure"
 		(shape input)
-		(at 212.725 92.71 0)
+		(at 221.234 92.71 0)
 		(fields_autoplaced yes)
 		(effects
@@
 				(path "/d5adb002-6fc2-438b-bcfe-09361e17acf4"
 					(reference "#PWR0104")
-					(unit 1)
-				)
-			)
-		)
-	)
-	(symbol
-		(lib_id "Device:R")
-		(at 206.629 92.71 90)
-		(unit 1)
-		(exclude_from_sim no)
-		(in_bom yes)
-		(on_board yes)
-		(dnp no)
-		(property "Reference" "R107"
-			(at 207.899 94.615 0)
-			(effects
-				(font
-					(size 1.27 1.27)
-				)
-				(justify right)
-			)
-		)
-		(property "Value" "10k"
-			(at 205.359 94.615 0)
-			(effects
-				(font
-					(size 1.27 1.27)
-				)
-				(justify right)
-			)
-		)
-		(property "Footprint" "Resistor_SMD:R_0402_1005Metric"
-			(at 206.629 94.488 90)
-			(effects
-				(font
-					(size 1.27 1.27)
-				)
-				(hide yes)
-			)
-		)
-		(property "Datasheet" "~"
-			(at 206.629 92.71 0)
-			(effects
-				(font
-					(size 1.27 1.27)
-				)
-				(hide yes)
-			)
-		)
-		(property "Description" ""
-			(at 206.629 92.71 0)
-			(effects
-				(font
-					(size 1.27 1.27)
-				)
-				(hide yes)
-			)
-		)
-		(property "LCSC" "C25744"
-			(at 206.629 92.71 0)
-			(effects
-				(font
-					(size 1.27 1.27)
-				)
-				(hide yes)
-			)
-		)
-		(pin "1"
-		)
-		(pin "2"
-		)
-		(instances
-			(project "TankPressure"
-				(path "/d5adb002-6fc2-438b-bcfe-09361e17acf4"
-					(reference "R107")
 					(unit 1)
 				)
@@
 	)
 	(symbol
+		(lib_id "Device:R")
+		(at 216.154 92.71 90)
+		(unit 1)
+		(exclude_from_sim no)
+		(in_bom yes)
+		(on_board yes)
+		(dnp no)
+		(property "Reference" "R107"
+			(at 216.154 88.9 90)
+			(effects
+				(font
+					(size 1.27 1.27)
+				)
+			)
+		)
+		(property "Value" "1k"
+			(at 216.154 90.805 90)
+			(effects
+				(font
+					(size 1.27 1.27)
+				)
+			)
+		)
+		(property "Footprint" "Resistor_SMD:R_0402_1005Metric"
+			(at 216.154 94.488 90)
+			(effects
+				(font
+					(size 1.27 1.27)
+				)
+				(hide yes)
+			)
+		)
+		(property "Datasheet" "~"
+			(at 216.154 92.71 0)
+			(effects
+				(font
+					(size 1.27 1.27)
+				)
+				(hide yes)
+			)
+		)
+		(property "Description" ""
+			(at 216.154 92.71 0)
+			(effects
+				(font
+					(size 1.27 1.27)
+				)
+				(hide yes)
+			)
+		)
+		(property "LCSC" " C11702"
+			(at 216.154 92.71 0)
+			(effects
+				(font
+					(size 1.27 1.27)
+				)
+				(hide yes)
+			)
+		)
+		(pin "1"
+		)
+		(pin "2"
+		)
+		(instances
+			(project "TankPressure"
+				(path "/d5adb002-6fc2-438b-bcfe-09361e17acf4"
+					(reference "R107")
+					(unit 1)
+				)
+			)
+		)
+	)
+	(symbol
 		(lib_id "Device:C")
 		(at 100.584 94.361 0)
@@
 			)
 		)
-		(property "Value" "L"
+		(property "Value" "1.5uH"
 			(at 124.079 63.246 90)
 			(effects
