File: hardware/modules/Rocket/LiPoPower2.kicad_sch (KiCad schematic)
At the start: 42 parts, among them J4 Ext Switch, J5 LiPo, U5 MCP73871-1CC, U6 INA226, U7 INA226, U8 TPS63070RNMR, U9 INA226

Commit message: ロケット電装回路図更新
Parts:
- added R12: 10k, Resistor_SMD:R_0402_1005Metric, symbol Device:R
Connections:
- net GND: now also R12.2
- net VDD_BUS: no longer C19.1, C7.1, U6.2 (A0), U6.6 (VS), U9.6 (VS)
- net at C8.1, R26.1, U5.1 (OUT)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: no longer C12.1, U7.6 (VS)
- net at U5.5 (THERM): now also R12.1
- new net: C12.1, C7.1, U6.2 (A0), U6.6 (VS), U7.6 (VS)
- new net: C19.1, U9.6 (VS)

Commit message: Rocket電装配置
Parts:
- added C105: 10uF, Capacitor_SMD:C_0603_1608Metric, symbol Device:C
- added J101: Conn_01x03, Connector_PinHeader_2.54mm:PinHeader_1x03_P2.54mm_Vertical, symbol Connector_Generic:Conn_01x03
- added R110: 4.7k, Resistor_SMD:R_0402_1005Metric, symbol Device:R
- added R112: 10k, Resistor_SMD:R_0402_1005Metric, symbol Device:R
- added U103: TPS2116DRL, Package_TO_SOT_SMD:SOT-583-8, symbol Power_Management:TPS2116DRL
- renumbered C6 to C104, C7 to C106, C10 to C107, C11 to C108, C8 to C109, C9 to C110, C13 to C111, C12 to C112, C14 to C113, C15 to C114, C16 to C115, C17 to C116, C18 to C117, C19 to C118, F2 to F101, F4 to F102, J4 to J102, J5 to J103, L2 to L101, LED2 to LED101, LED3 to LED102, LED6 to LED103, R9 to R108, R10 to R109, R11 to R111, R12 to R113, R14 to R114, R16 to R115, R26 to R116, R27 to R117, R28 to R118, R29 to R119, R30 to R120, R31 to R121, R32 to R122, R33 to R123, R34 to R124, RV2 to RV101, U5 to U104, U6 to U105, U7 to U106, U8 to U107, U9 to U108
Connections:
- net GND: now also C105.2, J101.3 (Pin_3), R110.1, U103.1 (GND)
- net VBUS: now also J101.1 (Pin_1)
- net VDD_BUS: now also C106.1, C112.1, C118.1, U105.2 (A0), U105.6 (VS), U106.6 (VS), U108.6 (VS)
- net at C109.1, U104.1 (OUT), U104.20 (OUT): now also C105.1, R112.1, U103.3 (VIN1), U103.5 (MODE); no longer R116.1, U105.10 (Vin+), U105.8 (Vbus)
- new net: R110.2, R112.2, U103.4 (PR1)
- new net: R116.1, U103.2 (VOUT), U103.7 (VOUT), U105.10 (Vin+), U105.8 (Vbus)
- new net DetLaunch: J101.2 (Pin_2)
- new net ST: U103.8 (ST)
Other:
- moved on the sheet: C104, C109, C110, C112, F101, F102, J103, LED101, LED102, R108, R109, R111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

Commit message: ロケット電装修正
Parts:
- added D301: D, Diode_SMD:D_SOD-323, symbol Device:D
Connections:
- net VBUS: now also D301.1 (K); no longer J101.1 (Pin_1)
- net VDD_BUS: no longer C106.1, C112.1, U105.2 (A0), U105.6 (VS), U106.6 (VS)
- net VPP: now reaches R116.1, U103.2 (VOUT), U103.7 (VOUT), U105.10 (Vin+), U105.8 (Vbus)
- net VPP: now also C106.1, C112.1, U105.2 (A0), U105.6 (VS), U106.6 (VS)
- new net: D301.2 (A), J101.1 (Pin_1)
Other:
- moved on the sheet: R116
