File: hardware/modules/Rocket/Rocket.kicad_pcb (KiCad board)
At the start: 2 copper layers, 93 parts, among them J101 Battery, J102 Temp&Heater, J103 Ext Switch, J104 LiPo, Q101 Q_NMOS_GSD, Q102 Q_NMOS_GSD, Q103 Q_PMOS_GSD, Q104 Q_PMOS_GSD, Q105 Q_PNP_BEC, Q106 Q_PNP_BEC, Q107 Q_PMOS_GSD, Q108 Q_NPN_BEC, Q109 Q_PMOS_GSD, SW101 Power Switch, SW2 RESET, U101 MCP73871-1CC, U102 INA226, U103 INA226, U104 TPS63070RNMR, U105 INA226, U2 TPS3820, U3 SN65HVD230, U4 ESP32-S3-WROOM-1

Commit message: 全て追加しました。
Parts:
- removed C101, C103, C104, C108, C110: 10uF, Capacitor_SMD:C_0603_1608Metric
- removed C102, C107, C109, C114: 100nF, Capacitor_SMD:C_0402_1005Metric
- removed C105, C106, C111, C112, C113: 22uF, Capacitor_SMD:C_0805_2012Metric
- removed D101: D_Schottky, Diode_SMD:D_SOD-323
- removed F101, F102, F103: Polyfuse, Fuse:Fuse_1206_3216Metric
- removed J101: Battery, Connector_JST:JST_XH_S2B-XH-A_1x02_P2.50mm_Horizontal
- removed J102: Temp&Heater, Connector_JST:JST_PH_S3B-PH-K_1x03_P2.00mm_Horizontal
- removed J103: Ext Switch, Connector_JST:JST_PH_S2B-PH-K_1x02_P2.00mm_Horizontal
- removed L101: L, Inductor_SMD:L_Wuerth_WE-TPC-3816
- removed LED101: USB Power, LED_SMD:LED_0603_1608Metric
- removed LED102: CHARGE, LED_SMD:LED_0603_1608Metric
- removed LED103: Backup Power, LED_SMD:LED_0603_1608Metric
- removed LED104: Heater, LED_SMD:LED_0603_1608Metric
- removed LED105: VDD, LED_SMD:LED_0603_1608Metric
- removed Q101, Q102: Q_NMOS_GSD, Package_TO_SOT_SMD:SOT-23-3
- removed Q103, Q104, Q107, Q109: Q_PMOS_GSD, Package_TO_SOT_SMD:SOT-23
- removed Q105, Q106: Q_PNP_BEC, Package_TO_SOT_SMD:SOT-23-3
- removed Q108: Q_NPN_BEC, Package_TO_SOT_SMD:SOT-23
- removed R101, R103, R107, R117, R126: 1k, PCM_Resistor_SMD_AKL:R_0402_1005Metric
- removed R104, R120, R124: 470k, PCM_Resistor_SMD_AKL:R_0402_1005Metric
- removed R105, R108, R109, R110, R112, R113, R114, R116, R122: 100k, PCM_Resistor_SMD_AKL:R_0402_1005Metric
- removed R111, R115, R119: 10k, PCM_Resistor_SMD_AKL:R_0402_1005Metric
- removed R118, R121, R125: 50mΩ, Resistor_SMD:R_0805_2012Metric
- removed R123: 150k, PCM_Resistor_SMD_AKL:R_0402_1005Metric
- removed RV101: 10k, PCM_Potentiometer_SMD_AKL:Potentiometer_Bourns_TC33X_Vertical
- removed SW101: Power Switch, Button_Switch_THT:SW_CuK_OS102011MA1QN1_SPDT_Angled
- removed U101: MCP73871-1CC, Package_DFN_QFN:QFN-20-1EP_4x4mm_P0.5mm_EP2.5x2.5mm
- removed U102, U103, U105: INA226, Package_SO:VSSOP-10_3x3mm_P0.5mm
- removed U104: TPS63070RNMR, WOBCLibrary:VREG_TPS63070RNMR
- added C10: 22uF, Capacitor_SMD:C_0805_2012Metric, F.Cu at (128.5, 76.3)
- added C11: 22uF, Capacitor_SMD:C_0805_2012Metric, F.Cu at (130.6, 76.3)
- added C12: 100nF, Capacitor_SMD:C_0402_1005Metric, F.Cu at (118.6, 75.4)
- added C120: 100p, Capacitor_SMD:C_0603_1608Metric, F.Cu at (217.1, 70.1)
- added C121: 100p, Capacitor_SMD:C_0603_1608Metric, F.Cu at (231.4, 70.2)
- added C122: 100n, Capacitor_SMD:C_0402_1005Metric, F.Cu at (222.9, 64.6)
- added C123: 100n, Capacitor_SMD:C_0402_1005Metric, F.Cu at (226.7, 64.6)
- added C124: 100p, Capacitor_SMD:C_0603_1608Metric, F.Cu at (224.8, 63.6)
- added C125: 10u, Capacitor_SMD:C_0603_1608Metric, F.Cu at (250.5, 41.1)
- added C126: 100n, Capacitor_SMD:C_0402_1005Metric, F.Cu at (249.3, 41.1)
- added C13: 10uF, Capacitor_SMD:C_0603_1608Metric, F.Cu at (133.1, 77.2)
- added C14: 100nF, Capacitor_SMD:C_0402_1005Metric, F.Cu at (137.6, 81.0)
- added C15: 10uF, Capacitor_SMD:C_0603_1608Metric, F.Cu at (136.0, 77.2)
- added C16: 22uF, Capacitor_SMD:C_0805_2012Metric, F.Cu at (138.6, 75.3)
- added C17: 22uF, Capacitor_SMD:C_0805_2012Metric, F.Cu at (139.3, 72.6)
- added C18: 22uF, Capacitor_SMD:C_0805_2012Metric, F.Cu at (141.3, 72.5)
- added C19: 100nF, Capacitor_SMD:C_0402_1005Metric, F.Cu at (144.4, 77.3)
- added C20: 10uF, Capacitor_SMD:C_0402_1005Metric, F.Cu at (194.0, 46.5)
- added C21: 100nF, Capacitor_SMD:C_0402_1005Metric, F.Cu at (194.0, 48.5)
- added C22: 100p, Capacitor_SMD:C_0603_1608Metric, F.Cu at (22.6, 26.3)
- added C23: 100p, Capacitor_SMD:C_0603_1608Metric, F.Cu at (22.6, 28.8)
- added C24: 100n, Capacitor_SMD:C_0402_1005Metric, F.Cu at (26.0, 26.0)
- added C25: 100n, Capacitor_SMD:C_0402_1005Metric, F.Cu at (26.0, 28.0)
- added C26: 100p, Capacitor_SMD:C_0603_1608Metric, F.Cu at (22.6, 31.3)
- added C27: 10u, Capacitor_SMD:C_0603_1608Metric, F.Cu at (22.6, 33.8)
- added C28: 100n, Capacitor_SMD:C_0402_1005Metric, F.Cu at (26.0, 30.0)
- added C29: 10μF, Capacitor_SMD:C_0603_1608Metric, F.Cu at (1.50, 0.76)
- added C29: 10μF, Capacitor_SMD:C_0402_1005Metric, F.Cu at (264.5, 81.1)
- added C30: 100nF, Capacitor_SMD:C_0402_1005Metric, F.Cu at (4.95, 0.48)
- added C30: 100nF, Capacitor_SMD:C_0402_1005Metric, F.Cu at (264.5, 83.1)
- added C31: 100nF, Capacitor_SMD:C_0402_1005Metric, F.Cu at (264.5, 85.0)
- added C31: 100nF, Capacitor_SMD:C_0402_1005Metric, F.Cu at (4.95, 2.46)
- added C32: 10μF, Capacitor_SMD:C_0603_1608Metric, F.Cu at (1.50, 3.27)
- added C32: 10μF, Capacitor_SMD:C_0402_1005Metric, F.Cu at (264.5, 87.0)
- added C33: 100nF, Capacitor_SMD:C_0402_1005Metric, F.Cu at (208.4, 134.6)
- added C34: 100nF, Capacitor_SMD:C_0402_1005Metric, F.Cu at (208.4, 136.6)
- added C35: 100nF, Capacitor_SMD:C_0402_1005Metric, F.Cu at (137.1, 156.7)
- added C36: 100nF, Capacitor_SMD:C_0402_1005Metric, F.Cu at (137.1, 158.7)
- added C37: 10μF, Capacitor_SMD:C_0603_1608Metric, F.Cu at (137.1, 160.7)
- added C38: 10μF, Capacitor_SMD:C_0603_1608Metric, F.Cu at (137.1, 162.7)
- added C39: 0.22μF, Capacitor_SMD:C_0402_1005Metric, F.Cu at (137.1, 164.6)
- added C40: 4.7μF, Capacitor_SMD:C_0603_1608Metric, F.Cu at (137.1, 166.6)
- added C41: 100nF, Capacitor_SMD:C_0402_1005Metric, F.Cu at (137.1, 168.6)
- added C42: 10μF, Capacitor_SMD:C_0603_1608Metric, F.Cu at (137.1, 170.5)
- added C6: 10uF, Capacitor_SMD:C_0603_1608Metric, F.Cu at (119.8, 79.7)
- added C7: 100nF, Capacitor_SMD:C_0402_1005Metric, F.Cu at (122.3, 74.0)
- added C8: 10uF, Capacitor_SMD:C_0603_1608Metric, F.Cu at (121.3, 79.7)
- added C9: 10uF, Capacitor_SMD:C_0603_1608Metric, F.Cu at (115.4, 75.4)
- added D10: ESD9B5.0ST5G, Diode_SMD:D_SOD-882, F.Cu at (213.8, 70.8)
- added D11: 5V, Diode_SMD:D_SOD-882D, F.Cu at (205.5, 134.8)
- added D12: 5V, Diode_SMD:D_SOD-882D, F.Cu at (205.5, 137.2)
- added D13: 5V, Diode_SMD:D_SOD-882D, F.Cu at (205.5, 139.5)
- added D8: D_Schottky, Diode_SMD:D_SOD-323, F.Cu at (105.2, 80.8)
- added D9: ESD9B5.0ST5G, Diode_SMD:D_SOD-882, F.Cu at (234.3, 70.9)
- added F2: Polyfuse, Fuse:Fuse_1206_3216Metric, F.Cu at (123.7, 97.5)
- added F3: Polyfuse, Fuse:Fuse_1206_3216Metric, F.Cu at (100.6, 74.2)
- added F4: Polyfuse, Fuse:Fuse_1206_3216Metric, F.Cu at (111.8, 73.2)
- added J105: SMA, Connector_Coaxial:SMA_Amphenol_132203-12_Horizontal, F.Cu at (234.0, 78.2)
- added J2: Battery, Connector_JST:JST_XH_S2B-XH-A_1x02_P2.50mm_Horizontal, F.Cu at (105.5, 69.0)
- added J3: Temp&Heater, Connector_JST:JST_PH_S3B-PH-K_1x03_P2.00mm_Horizontal, F.Cu at (130.5, 69.0)
- added J4: Ext Switch, Connector_JST:JST_PH_S2B-PH-K_1x02_P2.00mm_Horizontal, F.Cu at (141.5, 69.0)
- added J5: LiPo, Connector_JST:JST_PH_S2B-PH-K_1x02_P2.00mm_Horizontal, F.Cu at (117.5, 69.0)
- added J6: SMA, Connector_Coaxial:SMA_Amphenol_132203-12_Horizontal, F.Cu at (25.6, 20.0)
- added J7: SMA, Connector_Coaxial:SMA_Amphenol_132203-12_Horizontal, F.Cu at (35.6, 20.0)
- added J8: SMA, Connector_Coaxial:SMA_Amphenol_132203-12_Horizontal, F.Cu at (187.3, 135.9)
- added L2: L, Inductor_SMD:L_Wuerth_WE-TPC-3816, F.Cu at (134.5, 73.2)
- added L3: 27nH, 300mA, Inductor_SMD:L_0402_1005Metric, F.Cu at (208.7, 116.4)
- added LED2: USB Power, LED_SMD:LED_0805_2012Metric, F.Cu at (118.0, 98.0)
- added LED3: CHARGE, LED_SMD:LED_0805_2012Metric, F.Cu at (121.1, 69.0)
- added LED4: Backup Power, LED_SMD:LED_0805_2012Metric, F.Cu at (109.5, 69.0)
- added LED5: Heater, LED_SMD:LED_0805_2012Metric, F.Cu at (134.1, 69.0)
- added LED6: VDD, LED_SMD:LED_0805_2012Metric, F.Cu at (143.1, 72.5)
- added MICRO_SD2: TF-01A, WOBCLibrary:TF-01A, F.Cu at (189.0, 36.7)
- added Q10: Q_PMOS_GSD, Package_TO_SOT_SMD:SOT-23, F.Cu at (129.3, 72.5)
- added Q2: Q_NMOS_GSD, Package_TO_SOT_SMD:SOT-23-3, F.Cu at (103.8, 77.8)
- added Q3: Q_NMOS_GSD, Package_TO_SOT_SMD:SOT-23-3, F.Cu at (107.3, 77.8)
- added Q4: Q_PMOS_GSD, Package_TO_SOT_SMD:SOT-23, F.Cu at (103.8, 73.8)
- added Q5: Q_PMOS_GSD, Package_TO_SOT_SMD:SOT-23, F.Cu at (107.3, 73.8)
- added Q6: Q_PNP_BEC, Package_TO_SOT_SMD:SOT-23-3, F.Cu at (127.2, 80.2)
- added Q7: Q_PNP_BEC, Package_TO_SOT_SMD:SOT-23-3, F.Cu at (130.7, 80.2)
- added Q8: Q_PMOS_GSD, Package_TO_SOT_SMD:SOT-23, F.Cu at (123.8, 80.0)
- added Q9: Q_NPN_BEC, Package_TO_SOT_SMD:SOT-23, F.Cu at (125.4, 72.5)
- added R10: 1k, Resistor_SMD:R_0402_1005Metric, F.Cu at (123.5, 69.2)
- added R11: 1k, Resistor_SMD:R_0402_1005Metric, F.Cu at (113.3, 80.7)
- added R12: 470k, Resistor_SMD:R_0402_1005Metric, F.Cu at (101.5, 77.5)
- added R13: 100k, Resistor_SMD:R_0402_1005Metric, F.Cu at (100.4, 77.5)
- added R14: 100k, Resistor_SMD:R_0402_1005Metric, F.Cu at (117.6, 75.4)
- added R15: 1k, Resistor_SMD:R_0402_1005Metric, F.Cu at (112.4, 69.0)
- added R16: 100k, Resistor_SMD:R_0402_1005Metric, F.Cu at (113.3, 78.4)
- added R17: 100k, Resistor_SMD:R_0402_1005Metric, F.Cu at (101.0, 79.0)
- added R18: 100k, Resistor_SMD:R_0402_1005Metric, F.Cu at (109.6, 73.0)
- added R19: 10k, Resistor_SMD:R_0402_1005Metric, F.Cu at (107.9, 80.5)
- added R20: 100k, Resistor_SMD:R_0402_1005Metric, F.Cu at (107.9, 81.5)
- added R21: 100k, Resistor_SMD:R_0402_1005Metric, F.Cu at (124.5, 82.5)
- added R22: 100k, Resistor_SMD:R_0402_1005Metric, F.Cu at (122.5, 82.5)
- added R23: 10k, Resistor_SMD:R_0402_1005Metric, F.Cu at (122.3, 72.0)
- added R24: 100k, Resistor_SMD:R_0402_1005Metric, F.Cu at (122.3, 73.0)
- added R25: 1k, Resistor_SMD:R_0402_1005Metric, F.Cu at (136.5, 68.9)
- added R26: 50mΩ, Resistor_SMD:R_0805_2012Metric, F.Cu at (126.5, 76.3)
- added R27: 10k, Resistor_SMD:R_0402_1005Metric, F.Cu at (144.4, 81.8)
- added R28: 470k, Resistor_SMD:R_0402_1005Metric, F.Cu at (139.7, 80.6)
- added R29: 50mΩ, Resistor_SMD:R_0805_2012Metric, F.Cu at (113.9, 72.7)
- added R30: 100k, Resistor_SMD:R_0402_1005Metric, F.Cu at (134.5, 82.0)
- added R31: 150k, Resistor_SMD:R_0402_1005Metric, F.Cu at (137.6, 80.0)
- added R32: 470k, Resistor_SMD:R_0402_1005Metric, F.Cu at (137.6, 79.0)
- added R33: 50mΩ, Resistor_SMD:R_0805_2012Metric, F.Cu at (142.1, 75.3)
- added R34: 1k, Resistor_SMD:R_0402_1005Metric, F.Cu at (139.7, 78.5)
- added R35: 22k, Resistor_SMD:R_0402_1005Metric, F.Cu at (208.7, 118.4)
- added R36: 22k, Resistor_SMD:R_0402_1005Metric, F.Cu at (208.7, 120.4)
- added R37: 10, Resistor_SMD:R_0402_1005Metric, F.Cu at (208.7, 122.3)
- added R38: 33, Resistor_SMD:R_0402_1005Metric, F.Cu at (208.7, 124.3)
- added R39: 33, Resistor_SMD:R_0402_1005Metric, F.Cu at (208.7, 126.3)
- added R40: 4.7K, Resistor_SMD:R_0402_1005Metric, F.Cu at (140.0, 167.0)
- added R9: 1k, Resistor_SMD:R_0402_1005Metric, F.Cu at (120.7, 97.3)
- added RV2: 10k, Potentiometer_SMD:Potentiometer_Bourns_TC33X_Vertical, F.Cu at (110.9, 78.0)
- added SW3: Power Switch, Button_Switch_THT:SW_CuK_OS102011MA1QN1_SPDT_Angled, F.Cu at (148.8, 95.5)
- added Switch2: XA17-G4K1, Package_TO_SOT_SMD:SOT-363_SC-70-6, F.Cu at (224.8, 66.9)
- added U10: PCF8563T, Package_SO:SOIC-8_3.9x4.9mm_P1.27mm, F.Cu at (183.3, 48.9)
- added U107: E220-900T22S(JP), WOBCLibrary:E220-900T22S(JP), F.Cu at (238.8, 63.2)
- added U11: E220-900T22S(JP), WOBCLibrary:E220-900T22S(JP), F.Cu at (10.0, 25.1)
- added U12: ~, WOBClibraries:BME280, F.Cu at (267.9, 81.9)
- added U13: NEO-M9N-00B, WOBClibrary:SMT_9N-00B_UBL, F.Cu at (199.8, 124.5)
- added U14: BMI088, WOBClibraries:BMI088, F.Cu at (141.9, 159.1)
- added U15: QMC5883L, WOBClibraries:_HMC5883L, F.Cu at (140.7, 163.9)
- added U5: MCP73871-1CC, Package_DFN_QFN:QFN-20-1EP_4x4mm_P0.5mm_EP2.5x2.5mm, F.Cu at (116.5, 79.0)
- added U6: INA226, Package_SO:VSSOP-10_3x3mm_P0.5mm, F.Cu at (122.3, 76.3)
- added U7: INA226, Package_SO:VSSOP-10_3x3mm_P0.5mm, F.Cu at (118.1, 72.7)
- added U8: TPS63070RNMR, WOBCLibrary:VREG_TPS63070RNMR, F.Cu at (134.5, 79.7)
- added U9: INA226, Package_SO:VSSOP-10_3x3mm_P0.5mm, F.Cu at (142.1, 79.7)
- added USB3: USB_C_Receptacle_USB2.0, Connector_USB:USB_C_Receptacle_XKB_U262-16XN-4BVC11, F.Cu at (198.2, 138.9)
- added Y2: Crystal, Crystal:Crystal_SMD_3215-2Pin_3.2x1.5mm, F.Cu at (190.0, 47.2)
- J104: value LiPo -> SMA; footprint Connector_JST:JST_PH_S2B-PH-K_1x02_P2.00mm_Horizontal -> Connector_Coaxial:SMA_Amphenol_132203-12_Horizontal
- R102: value 1k -> 4.7K; footprint PCM_Resistor_SMD_AKL:R_0402_1005Metric -> Resistor_SMD:R_0402_1005Metric
- R106: value 100k -> 100K; footprint PCM_Resistor_SMD_AKL:R_0402_1005Metric -> Resistor_SMD:R_0402_1005Metric
- moved R102 101.6 mm to (140.0, 169.0), turned to 0 degrees
- moved R106 79.2 mm to (208.7, 128.3), turned to 0 degrees
- moved J104 64.8 mm to (214.1, 78.0)
Connections:
- J104 pad 1: Net-(J104-Pin_1) -> (no net)
- R102 pad 1: Net-(LED102-A) -> (no net)
- R102 pad 2: /LiPopower/CHARGE_IND -> (no net)
- R106 pad 1: Net-(U101-PROG3) -> (no net)
Routing:
- net Net-(U8-L1): track 0.00 -> 15.9 mm, vias 0 -> 7
- net Net-(U104-L1): track 15.9 -> 0.00 mm, vias 7 -> 0
- net Net-(U8-L2): track 0.00 -> 15.9 mm, vias 0 -> 7
- net Net-(U104-L2): track 15.9 -> 0.00 mm, vias 7 -> 0
- net Net-(D10-A2): track 0.00 -> 10.8 mm
- net Net-(D9-A2): track 0.00 -> 10.6 mm
- net Net-(Switch2-J3): track 0.00 -> 7.62 mm
- net Net-(Switch2-J2): track 0.00 -> 6.66 mm
- net (no net): track 0.00 -> 6.13 mm
- net Net-(U6-Vin-): track 0.00 -> 3.88 mm
- net Net-(U102-Vin-): track 3.88 -> 0.00 mm
- net VDD: track 0.00 -> 3.45 mm
- net /LoRa/RF_switch2: track 0.00 -> 1.65 mm
- net /LoRa/RF_switch1: track 0.00 -> 1.59 mm
- net Net-(Switch2-J1): track 0.00 -> 1.52 mm

Commit message: ロケット電装です
Parts:
- removed C120, C121, C124, C22, C23: 100p, Capacitor_SMD:C_0603_1608Metric
- removed C122, C123, C126, C24, C25: 100n, Capacitor_SMD:C_0402_1005Metric
- removed C125: 10u, Capacitor_SMD:C_0603_1608Metric
- removed the C29 at (1.50, 0.76)
- removed the C29 at (264.5, 81.1)
- removed C3, C41: 100nF, Capacitor_SMD:C_0402_1005Metric
- removed the C30 at (4.95, 0.48)
- removed the C30 at (264.5, 83.1)
- removed the C31 at (264.5, 85.0)
- removed the C31 at (4.95, 2.46)
- removed the C32 at (1.50, 3.27)
- removed the C32 at (264.5, 87.0)
- removed C42: 10μF, Capacitor_SMD:C_0603_1608Metric
- removed the C5 at (41.1, 48.3)
- removed the C5 at (60.3, 43.1)
- removed D11, D12, D13: 5V, Diode_SMD:D_SOD-882D
- removed D8: D_Schottky, Diode_SMD:D_SOD-323
- removed D9: ESD9B5.0ST5G, Diode_SMD:D_SOD-882
- removed F3: Polyfuse, Fuse:Fuse_1206_3216Metric
- removed J104, J105, J7: SMA, Connector_Coaxial:SMA_Amphenol_132203-12_Horizontal
- removed J2: Battery, Connector_JST:JST_XH_S2B-XH-A_1x02_P2.50mm_Horizontal
- removed J3: Temp&Heater, Connector_JST:JST_PH_S3B-PH-K_1x03_P2.00mm_Horizontal
- removed L3: 27nH, 300mA, Inductor_SMD:L_0402_1005Metric
- removed LED4: Backup Power, LED_SMD:LED_0805_2012Metric
- removed LED5: Heater, LED_SMD:LED_0805_2012Metric
- removed Q10, Q4, Q5, Q8: Q_PMOS_GSD, Package_TO_SOT_SMD:SOT-23
- removed Q2, Q3: Q_NMOS_GSD, Package_TO_SOT_SMD:SOT-23-3
- removed Q6, Q7: Q_PNP_BEC, Package_TO_SOT_SMD:SOT-23-3
- removed Q9: Q_NPN_BEC, Package_TO_SOT_SMD:SOT-23
- removed R102, R40: 4.7K, Resistor_SMD:R_0402_1005Metric
- removed R106: 100K, Resistor_SMD:R_0402_1005Metric
- removed R12: 470k, Resistor_SMD:R_0402_1005Metric
- removed R13, R17, R18, R20, R21, R22, R24: 100k, Resistor_SMD:R_0402_1005Metric
- removed R15, R25: 1k, Resistor_SMD:R_0402_1005Metric
- removed R19, R23: 10k, Resistor_SMD:R_0402_1005Metric
- removed R38, R39: 33, Resistor_SMD:R_0402_1005Metric
- removed SW3: Power Switch, Button_Switch_THT:SW_CuK_OS102011MA1QN1_SPDT_Angled
- removed Switch2: XA17-G4K1, Package_TO_SOT_SMD:SOT-363_SC-70-6
- removed U107: E220-900T22S(JP), WOBCLibrary:E220-900T22S(JP)
- removed U3: SN65HVD230, PCM_Package_TO_SOT_SMD_AKL:SOT-23-5
- removed USB3: USB_C_Receptacle_USB2.0, Connector_USB:USB_C_Receptacle_XKB_U262-16XN-4BVC11
- added C29: 10μF, Capacitor_SMD:C_0402_1005Metric, F.Cu at (269.0, 102.6)
- added C30: 100nF, Capacitor_SMD:C_0402_1005Metric, F.Cu at (269.0, 104.6)
- added C31: 100nF, Capacitor_SMD:C_0402_1005Metric, F.Cu at (269.0, 106.5)
- added C32: 10μF, Capacitor_SMD:C_0402_1005Metric, F.Cu at (269.0, 108.5)
- added C5: 100nF, Capacitor_SMD:C_0402_1005Metric, F.Cu at (65.1, 70.3)
- C35, C36: value 100nF -> 10μF; footprint Capacitor_SMD:C_0402_1005Metric -> Capacitor_SMD:C_0603_1608Metric
- C37: value 10μF -> 0.22μF; footprint Capacitor_SMD:C_0603_1608Metric -> Capacitor_SMD:C_0402_1005Metric
- C38: value 10μF -> 4.7μF
- C39: value 0.22μF -> 100nF
- C4: footprint Capacitor_SMD:C_0402_1005Metric -> Capacitor_SMD:C_0603_1608Metric
- C40: value 4.7μF -> 10μF
- D2, D3, D4: footprint Diode_SMD:D_SOD-923 -> Diode_SMD:D_SOD-882
- D5, D6, D7: footprint LED_SMD:LED_0603_1608Metric -> LED_SMD:LED_0805_2012Metric
- J6: value SMA -> Conn_01x02; footprint Connector_Coaxial:SMA_Amphenol_132203-12_Horizontal -> Connector_PinHeader_1.00mm:PinHeader_1x02_P1.00mm_Vertical
- R28: value 470k -> 330k
- R31: value 150k -> 15k
- R32: value 470k -> 47k
- R35, R36: value 22k -> 470
- R37: value 10 -> 4.7K
- SW2: value RESET -> RESET_sw
- U11: value E220-900T22S(JP) -> SAM-M10Q; footprint WOBCLibrary:E220-900T22S(JP) -> RF_GPS:ublox_SAM-M8Q
- U12: value ~ -> E220-900T22S(JP); footprint WOBClibraries:BME280 -> WOBCLibrary:E220-900T22S(JP)
- U13: value NEO-M9N-00B -> ~; footprint WOBClibrary:SMT_9N-00B_UBL -> WOBClibraries:BME280
- U2: footprint RF_Module:ESP32-S3-WROOM-1 -> PCM_Package_TO_SOT_SMD_AKL:SOT-23-5; moved to F.Cu
- U4: footprint Package_SO:SOIC-8_3.9x4.9mm_P1.27mm -> RF_Module:ESP32-S3-WROOM-1; moved to B.Cu
- moved C27 261.1 mm to (283.5, 23.6), turned to 90 degrees
- moved C28 256.4 mm to (282.3, 23.6), turned to 90 degrees
- moved C26 235.7 mm to (257.8, 46.1), turned to -90 degrees
- moved U11 231.5 mm to (226.9, 106.0)
- moved J6 230.5 mm to (240.0, 104.5)
- moved U14 122.2 mm to (255.9, 115.1)
- moved U15 122.2 mm to (254.7, 119.9)
- moved C35 120.8 mm to (251.1, 116.7)
- moved C36 120.8 mm to (251.1, 118.7)
- moved C37 120.8 mm to (251.1, 120.6)
- moved C38 120.8 mm to (251.1, 122.6)
- moved C39 120.8 mm to (251.1, 124.6)
- moved C40 120.8 mm to (251.1, 126.5)
- moved J8 109.5 mm to (267.0, 60.8), turned to 180 degrees
- moved U13 75.6 mm to (272.4, 103.4)
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Connections:
- net /9DoF/I2C_SCL renamed /9DoF2/I2C_SCL
- net /9DoF/I2C_SDA renamed /9DoF2/I2C_SDA
- net /ESP32Core/GPIO4/ADC1_CH3 renamed /ESP32Core2/GPIO4/ADC1_CH3
- net /ESP32Core/GPIO5/ADC1_CH4 renamed /ESP32Core2/GPIO5/ADC1_CH4
- net /ESP32Core/GPIO6/ADC1_CH5 renamed /ESP32Core2/GPIO6/ADC1_CH5
- net /ESP32Core/GPIO7/ADC1_CH6 renamed /ESP32Core2/GPIO7/ADC1_CH6
- net /ESP32Core/VUSB renamed /ESP32Core2/VUSB
- net /ESP32Core/WDI renamed /ESP32Core2/WDI
- net /GPSActive/TIMEPULSE renamed /Pressure2/I2C_SDA
- net /LiPopower/CHARGE_IND renamed /LiPoPower2/CHARGE_IND
- net /LiPopower/I2C_SCL renamed /LiPoPower2/I2C_SCL
- net /LiPopower/I2C_SDA renamed /LiPoPower2/I2C_SDA
- net /LiPopower/PG renamed /LiPoPower2/PG
- net /LiPopower/PROG renamed /LiPoPower2/PROG
- net /LiPopower/STAT1 renamed /LiPoPower2/STAT1
- net /LiPopower/STAT2 renamed /LiPoPower2/STAT2
- net /LiPopower/VDD_BUS renamed /LiPoPower2/VDD_BUS
- net /LoRa/LoRa_TRX renamed /GPS SAM-M10Q2/TIME PULSE
- net /Logger/I2C_SCL renamed /Logger2/I2C_SCL
- net /Logger/I2C_SDA renamed /Logger2/I2C_SDA
- net /Logger/SD_CLK renamed /Logger2/SD_CLK
- net /Logger/SD_DET renamed /Logger2/SD_DET
- net /Logger/SD_MISO renamed /Logger2/SD_MISO
- net /Logger/SD_MOSI renamed /Logger2/SD_MOSI
- net /Logger/SD_SS renamed /Logger2/SD_SS
- C12 pad 1: Net-(Q3-G) -> Net-(U6-Vbus)
- C26 pad 1: Net-(U11-ANT) -> Net-(U12-ANT)
- C26 pad 2: Net-(Switch2-J1) -> Net-(D10-A2)
- C33 pad 1: Net-(C33-Pad1) -> VDD
- C34 pad 1: GND -> VDD
- C34 pad 2: VDD -> GND
- C37 pad 1: VDD -> Net-(U15-SETC)
- C37 pad 2: GND -> Net-(U15-STEP)
- C38 pad 1: VDD -> Net-(U15-C1)
- C39 pad 1: Net-(U15-SETC) -> VDD
- C39 pad 2: Net-(U15-STEP) -> GND
- C40 pad 1: Net-(U15-C1) -> VDD
- C8 pad 1: Net-(Q3-G) -> Net-(U6-Vbus)
- D3 pad 2: /ESP32Core/USB_D+ -> /ESP32Core2/USB_D+
- D4 pad 2: /ESP32Core/USB_D- -> /ESP32Core2/USB_D-
- J6 pad 1: Net-(D9-A2) -> /GPS SAM-M10Q2/RX
- J6 pad 2: GND -> /GPS SAM-M10Q2/TX
- J8 pad 1: GPS_ANT1 -> Net-(D10-A2)
- R26 pad 1: VPP -> Net-(U6-Vbus)
- R35 pad 1: Net-(USB3-CC1) -> Net-(U11-TXD)
- R35 pad 2: GND -> /GPS SAM-M10Q2/TX
- R36 pad 1: Net-(USB3-CC2) -> Net-(U11-RXD)
- R36 pad 2: GND -> /GPS SAM-M10Q2/RX
- R37 pad 1: VCC_RF -> Net-(U14-SDO1)
- R37 pad 2: Net-(C33-Pad1) -> VDD
- R6 pad 2: /ESP32Core/I2C_SCL -> /ESP32Core2/I2C_SCL
- R8 pad 2: /ESP32Core/I2C_SDA -> /ESP32Core2/I2C_SDA
- U11 pad 10: VDD -> GND
- U11 pad 12: (no net) -> unconnected-(U11-SCL-Pad12)
- U11 pad 13: GND -> Net-(U11-TXD)
- U11 pad 14: (no net) -> Net-(U11-RXD)
- U11 pad 15: (no net) -> GND
- U11 pad 16: (no net) -> GND
- U11 pad 17: (no net) -> VDD
- U11 pad 18: (no net) -> /GPS SAM-M10Q2/RESET
- U11 pad 19: GND -> unconnected-(U11-EXTINT-Pad19)
- U11 pad 2: GND -> VDD
- U11 pad 3: GND -> /GPS SAM-M10Q2/BUCKUP
- U11 pad 5: /LoRa/LoRa_M0 -> GND
- U11 pad 6: /LoRa/LoRa_M1 -> GND
- U11 pad 8: /LoRa/LoRa_RTX -> unconnected-(U11-~{SAFEBOOT}-Pad8)
- U11 pad 9: /LoRa/LoRa_AUX -> unconnected-(U11-SDA-Pad9)
- U12 pad 2: VDD -> GND
- U12 pad 3: /Pressure/I2C_SDA -> GND
- U12 pad 4: /Pressure/I2C_SCL -> GND
- U12 pad 5: GND -> /LoRa2/LoRa_M0
- U12 pad 6: VDD -> /LoRa2/LoRa_M1
- U12 pad 7: GND -> /LoRa2/LoRa_TRX
- U12 pad 8: VDD -> /LoRa2/LoRa_RTX
- U13 pad 1: unconnected-(U13-SAFEBOOT_N-Pad1) -> GND
- U13 pad 2: unconnected-(U13-D_SEL-Pad2) -> VDD
- U13 pad 4: unconnected-(U13-EXTINT-Pad4) -> /Pressure2/I2C_SCL
- U13 pad 5: /GPSActive/USB_D- -> GND
- U13 pad 6: /GPSActive/USB_D+ -> VDD
- U13 pad 7: VDD -> GND
- U13 pad 8: /GPSActive/RESET -> VDD
- U5 pad 1: Net-(Q3-G) -> Net-(U6-Vbus)
- U5 pad 20: Net-(Q3-G) -> Net-(U6-Vbus)
- U5 pad 5: /LiPopower/TEMP -> unconnected-(U5-THERM-Pad5)
- U6 pad 10: VPP -> Net-(U6-Vbus)
- U6 pad 8: VPP -> Net-(U6-Vbus)
- U7 pad 6: Net-(Q3-G) -> Net-(U6-Vbus)
- USB2 pad A6: /ESP32Core/USB_D+ -> /ESP32Core2/USB_D+
- USB2 pad A7: /ESP32Core/USB_D- -> /ESP32Core2/USB_D-
- USB2 pad B6: /ESP32Core/USB_D+ -> /ESP32Core2/USB_D+
- USB2 pad B7: /ESP32Core/USB_D- -> /ESP32Core2/USB_D-
Routing:
- net Net-(D9-A2): track 10.6 -> 0.00 mm
- net Net-(Switch2-J3): track 7.62 -> 0.00 mm
- net Net-(Switch2-J2): track 6.66 -> 0.00 mm
- net Net-(U12-ANT): track 0.00 -> 6.13 mm
- net (no net): track 6.13 -> 3.24 mm
- net /LoRa/RF_switch2: track 1.65 -> 0.00 mm
- net /LoRa/RF_switch1: track 1.59 -> 0.00 mm
- net Net-(Switch2-J1): track 1.52 -> 0.00 mm
- net Net-(D10-A2): track 10.8 -> 12.1 mm
Other:
- board outline added: 100 x 35 mm

Commit message: ロケット電装回路図更新
Parts:
- added R12: 10k, Resistor_SMD:R_0402_1005Metric, F.Cu at (115.6, 168.8)
- J8: value SMA -> UFL; footprint Connector_Coaxial:SMA_Amphenol_132203-12_Horizontal -> Connector_Coaxial:U.FL_Molex_MCRF_73412-0110_Vertical
- R35: value 470 -> 470
- U11, U12: moved to B.Cu
- moved C27 177.8 mm to (126.5, 107.0)
- moved C28 177.8 mm to (125.3, 107.0)
- moved J8 155.7 mm to (120.5, 113.5), turned to 0 degrees
- moved U12 153.4 mm to (132.1, 109.0), turned to -90 degrees
- moved C26 150.7 mm to (118.2, 103.1)
- moved D10 150.7 mm to (127.8, 110.4)
- moved J6 139.9 mm to (102.1, 80.8)
- moved R35 139.9 mm to (99.0, 82.5)
- moved R36 139.9 mm to (99.0, 80.5)
- moved U13 138.6 mm to (134.4, 90.9)
- moved C29 138.6 mm to (131.0, 90.0)
- moved C30 138.6 mm to (131.0, 92.0)
- moved C31 138.6 mm to (131.0, 94.0)
- moved C32 138.6 mm to (131.0, 95.9)
- moved C33 130.1 mm to (125.3, 79.6)
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Connections:
- C12 pad 1: Net-(U6-Vbus) -> Net-(U6-A0)
- C19 pad 1: /LiPoPower2/VDD_BUS -> Net-(U9-VS)
- C7 pad 1: /LiPoPower2/VDD_BUS -> Net-(U6-A0)
- U5 pad 5: unconnected-(U5-THERM-Pad5) -> Net-(U5-THERM)
- U6 pad 2: /LiPoPower2/VDD_BUS -> Net-(U6-A0)
- U6 pad 6: /LiPoPower2/VDD_BUS -> Net-(U6-A0)
- U7 pad 6: Net-(U6-Vbus) -> Net-(U6-A0)
- U9 pad 6: /LiPoPower2/VDD_BUS -> Net-(U9-VS)
Routing:
- net Net-(D10-A2): track 12.1 -> 0.00 mm
- net GND: track 22.1 -> 13.3 mm
- net Net-(U12-ANT): track 6.13 -> 0.00 mm
- net Net-(U6-Vin-): track 3.88 -> 0.23 mm
- net VDD: track 3.45 -> 0.01 mm
- net Net-(U8-L2): track 15.9 -> 12.5 mm
- net (no net): track 3.24 -> 0.00 mm
Other:
- board size 100 x 35 mm -> 35 x 100 mm

Commit message: Rocket電装配置
Parts:
- removed J6: Conn_01x02, Connector_PinHeader_1.00mm:PinHeader_1x02_P1.00mm_Vertical
- added ?: , , F.Cu at (137.5, 47.0)
- added ?: , , F.Cu at (137.5, 146.0)
- added BT101: Battery_Cell, WOBCLibrary:cr1220, B.Cu at (132.4, 61.7)
- added C105: 10uF, Capacitor_SMD:C_0603_1608Metric, F.Cu at (145.2, 109.5)
- added J101: Conn_01x03, Connector_PinHeader_2.54mm:PinHeader_1x03_P2.54mm_Vertical, F.Cu at (122.5, 108.5)
- added J104: Conn_01x02, Connector_PinHeader_2.54mm:PinHeader_1x02_P2.54mm_Vertical, F.Cu at (121.9, 61.8)
- added R110: 4.7k, Resistor_SMD:R_0402_1005Metric, F.Cu at (140.4, 109.2)
- added R112: 10k, Resistor_SMD:R_0402_1005Metric, F.Cu at (140.9, 110.8)
- added SW102: SW_Push_DPDT, WOBCLibrary:IS-2245S-G, F.Cu at (128.8, 60.7)
- added U103: TPS2116DRL, Package_TO_SOT_SMD:SOT-583-8, F.Cu at (142.3, 108.9)
- R101: renamed from R2; value 22k -> 5.1k
- R102: renamed from R3; value 22k -> 5.1k
- U110: renamed from U11; moved to F.Cu
- moved J103 73.1 mm to (152.7, 116.0), turned to 90 degrees
- moved F102 71.7 mm to (149.6, 114.8), turned to -90 degrees
- moved R119 70.8 mm to (145.7, 111.5), turned to 0 degrees
- moved J102 68.6 mm to (153.3, 103.8), turned to 90 degrees
- moved LED102 67.0 mm to (123.2, 99.1), turned to 90 degrees
- moved R120 66.7 mm to (150.8, 99.5)
- moved C108 66.5 mm to (148.5, 104.5)
- moved R109 65.4 mm to (125.6, 99.2), turned to 90 degrees
- moved C112 65.3 mm to (148.0, 113.2), turned to 90 degrees
- moved C102 65.1 mm to (125.3, 76.3), turned to -90 degrees
- moved C113 65.1 mm to (149.9, 98.4)
- moved R121 65.1 mm to (148.9, 98.4)
- moved R122 65.1 mm to (147.9, 98.4)
- moved U107 65.1 mm to (148.6, 101.4)
- moved R118 64.7 mm to (152.4, 98.8)
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- renumbered C2 to C101, C4 to C102, C5 to C103, C6 to C104, C7 to C106, C10 to C107, C11 to C108, C8 to C109, C9 to C110, C13 to C111, C12 to C112, C14 to C113, C15 to C114, C16 to C115, C17 to C116, C18 to C117, C19 to C118, C20 to C119, C21 to C120, C26 to C121, C27 to C122, C28 to C123, C29 to C124, C30 to C125, C31 to C126, C32 to C127, C33 to C128, C34 to C129, C35 to C130, C36 to C131, C37 to C132, C38 to C133, C39 to C134, C40 to C135, D2 to D101, D3 to D102, D4 to D103, D5 to D104, D6 to D105, D7 to D106, D10 to D107, F2 to F101, F4 to F102, J4 to J102, J5 to J103, J8 to J105, L2 to L101, LED2 to LED101, LED3 to LED102, LED6 to LED103, MICRO_SD2 to MICRO_SD101, R4 to R103, R5 to R104, R6 to R105, R7 to R106, R8 to R107, R9 to R108, R10 to R109, R11 to R111, R12 to R113, R14 to R114, R16 to R115, R26 to R116, R27 to R117, R28 to R118, R29 to R119, R30 to R120, R31 to R121, R32 to R122, R33 to R123, R34 to R124, R36 to R125, R35 to R126, R37 to R127, RV2 to RV101, SW2 to SW101, U2 to U101, U4 to U102, U5 to U104, U6 to U105, U7 to U106, U8 to U107, U9 to U108, U10 to U109, U12 to U111, U13 to U112, U14 to U113, U15 to U114, USB2 to USB101, Y2 to Y101
Connections:
- C106 pad 1: Net-(U6-A0) -> VBUS
- C109 pad 1: Net-(U6-Vbus) -> Net-(U103-MODE)
- C112 pad 1: Net-(U6-A0) -> VBUS
- C114 pad 1: /LiPoPower2/VDD_BUS -> VBUS
- C115 pad 1: /LiPoPower2/VDD_BUS -> VBUS
- C116 pad 1: /LiPoPower2/VDD_BUS -> VBUS
- C117 pad 1: /LiPoPower2/VDD_BUS -> VBUS
- C118 pad 1: Net-(U9-VS) -> VBUS
- D101 pad 2: /ESP32Core2/VUSB -> VBUS
- MICRO_SD101 pad 2: /Logger2/SD_SS -> /SS
- MICRO_SD101 pad 3: /Logger2/SD_MOSI -> /MOSI
- MICRO_SD101 pad 5: /Logger2/SD_CLK -> /CLK
- MICRO_SD101 pad 7: /Logger2/SD_MISO -> /MISO
- MICRO_SD101 pad CD1: /Logger2/SD_DET -> /SD_DET
- R105 pad 2: /ESP32Core2/I2C_SCL -> /I2C_SCL
- R107 pad 2: /ESP32Core2/I2C_SDA -> /I2C_SDA
- R109 pad 2: /LiPoPower2/CHARGE_IND -> /CHARGE
- R116 pad 1: Net-(U6-Vbus) -> Net-(U105-Vbus)
- R120 pad 1: /LiPoPower2/VDD_BUS -> VBUS
- R122 pad 2: /LiPoPower2/VDD_BUS -> VBUS
- R123 pad 1: /LiPoPower2/VDD_BUS -> VBUS
- R125 pad 2: /GPS SAM-M10Q2/RX -> Net-(R125-Pad2)
- R126 pad 2: /GPS SAM-M10Q2/TX -> Net-(R126-Pad2)
- U102 pad 10: /ESP32Core2/I2C_SDA -> /I2C_SDA
- U102 pad 11: /ESP32Core2/GPIO18 -> /TimePulse
- U102 pad 12: /ESP32Core2/GPIO8/ADC1_CH7 -> /GPS_RESET
- U102 pad 15: /ESP32Core2/GPIO3/ADC1_CH2 -> /MISO
- U102 pad 20: /ESP32Core2/GPIO12 -> /DetL
- U102 pad 21: /ESP32Core2/GPIO13 -> /ST
- U102 pad 22: /ESP32Core2/GPIO14 -> /CHARGE
- U102 pad 23: /ESP32Core2/GPIO21 -> /PG
- U102 pad 24: /ESP32Core2/GPIO47 -> /STAT1
- U102 pad 25: /ESP32Core2/GPIO48 -> /STAT2
- U102 pad 31: /ESP32Core2/GPIO38 -> /AUX
- U102 pad 32: /ESP32Core2/GPIO39 -> /M0
- U102 pad 33: /ESP32Core2/GPIO40 -> /M1
- U102 pad 36: /ESP32Core2/CAN_RX -> /RTX0
- U102 pad 37: /ESP32Core2/CAN_TX -> /TRX0
- U102 pad 38: /ESP32Core2/GPIO2/ADC1_CH1 -> /SS
- U102 pad 39: /ESP32Core2/GPIO1/ADC1_CH0 -> /CLK
- U102 pad 4: /ESP32Core2/GPIO4/ADC1_CH3 -> /MOSI
- U102 pad 5: /ESP32Core2/GPIO5/ADC1_CH4 -> /SD_DET
- U102 pad 6: /ESP32Core2/GPIO6/ADC1_CH5 -> /TRX1
- U102 pad 7: /ESP32Core2/GPIO7/ADC1_CH6 -> /RTX1
- U102 pad 9: /ESP32Core2/I2C_SCL -> /I2C_SCL
- U104 pad 1: Net-(U6-Vbus) -> Net-(U103-MODE)
- U104 pad 20: Net-(U6-Vbus) -> Net-(U103-MODE)
- U104 pad 6: /LiPoPower2/PG -> /PG
- U104 pad 7: /LiPoPower2/STAT2 -> /STAT2
- U104 pad 8: /LiPoPower2/STAT1 -> /STAT1
- U105 pad 1: /LiPoPower2/I2C_SCL -> /I2C_SCL
- U105 pad 10: Net-(U6-Vbus) -> Net-(U105-Vbus)
- U105 pad 2: Net-(U6-A0) -> VBUS
- U105 pad 4: /LiPoPower2/I2C_SDA -> /I2C_SDA
- U105 pad 5: /LiPoPower2/I2C_SCL -> /I2C_SCL
- U105 pad 6: Net-(U6-A0) -> VBUS
- U105 pad 8: Net-(U6-Vbus) -> Net-(U105-Vbus)
- U106 pad 1: /LiPoPower2/I2C_SCL -> /I2C_SCL
- U106 pad 2: /LiPoPower2/I2C_SCL -> /I2C_SCL
- U106 pad 4: /LiPoPower2/I2C_SDA -> /I2C_SDA
- U106 pad 5: /LiPoPower2/I2C_SCL -> /I2C_SCL
- U106 pad 6: Net-(U6-A0) -> VBUS
- U107 pad 7_8: /LiPoPower2/VDD_BUS -> VBUS
- U108 pad 1: /LiPoPower2/I2C_SCL -> /I2C_SCL
- U108 pad 10: /LiPoPower2/VDD_BUS -> VBUS
- U108 pad 2: /LiPoPower2/I2C_SDA -> /I2C_SDA
- U108 pad 4: /LiPoPower2/I2C_SDA -> /I2C_SDA
- U108 pad 5: /LiPoPower2/I2C_SCL -> /I2C_SCL
- U108 pad 6: Net-(U9-VS) -> VBUS
- U108 pad 8: /LiPoPower2/VDD_BUS -> VBUS
- U109 pad 5: /Logger2/I2C_SDA -> /I2C_SDA
- U109 pad 6: /Logger2/I2C_SCL -> /I2C_SCL
- U110 pad 18: /GPS SAM-M10Q2/RESET -> /GPS_RESET
- U110 pad 7: /GPS SAM-M10Q2/TIME PULSE -> /TimePulse
- U111 pad 5: /LoRa2/LoRa_M0 -> /M0
- U111 pad 6: /LoRa2/LoRa_M1 -> /M1
- U111 pad 7: /LoRa2/LoRa_TRX -> /TRX0
- U111 pad 8: /LoRa2/LoRa_RTX -> /RTX0
- U111 pad 9: /LoRa2/LoRa_AUX -> /AUX
- U112 pad 3: /Pressure2/I2C_SDA -> /I2C_SDA
- U112 pad 4: /Pressure2/I2C_SCL -> /I2C_SCL
- U113 pad 8: /9DoF2/I2C_SCL -> /I2C_SCL
- U113 pad 9: /9DoF2/I2C_SDA -> /I2C_SDA
- U114 pad 1: /9DoF2/I2C_SCL -> /I2C_SCL
- U114 pad 16: /9DoF2/I2C_SDA -> /I2C_SDA
- USB101 pad A4: /ESP32Core2/VUSB -> VBUS
- USB101 pad A9: /ESP32Core2/VUSB -> VBUS
- USB101 pad B4: /ESP32Core2/VUSB -> VBUS
- USB101 pad B9: /ESP32Core2/VUSB -> VBUS
Routing:
- net GND: track 13.3 -> 0.07 mm
- net /LiPoPower2/VDD_BUS: track 9.88 -> 0.00 mm
- net Net-(U107-L1): track 15.9 -> 7.90 mm, vias 7 -> 5
- net Net-(U107-L2): track 12.5 -> 7.90 mm, vias 7 -> 5
Other:
- board size 35 x 100 mm -> 35 x 107 mm

Commit message: 配線途中です
Parts:
- moved D107 1.15 mm to (121.7, 136.5)
Routing:
- net VDD: track 0.00 -> 174.9 mm, vias 0 -> 3
- net /I2C_SDA: track 0.00 -> 97.1 mm, vias 0 -> 8
- net /I2C_SCL: track 0.00 -> 91.8 mm, vias 0 -> 2
- net /SD_DET: track 0.00 -> 69.1 mm, vias 0 -> 3
- net /MISO: track 0.00 -> 61.7 mm, vias 0 -> 2
- net /MOSI: track 0.00 -> 60.5 mm, vias 0 -> 2
- net /CLK: track 0.00 -> 45.8 mm, vias 0 -> 5
- net /SS: track 0.00 -> 45.1 mm, vias 0 -> 3
- net /CHARGE: track 0.00 -> 26.5 mm
- net /TimePulse: track 0.00 -> 26.5 mm
- net /GPS_RESET: track 0.00 -> 21.8 mm, vias 0 -> 1
- net /RTX1: track 0.00 -> 7.46 mm, vias 0 -> 2
- net /ESP32Core2/USB_D-: track 0.00 -> 6.53 mm, vias 0 -> 1
- net /ESP32Core2/USB_D+: track 0.00 -> 5.33 mm
- net Net-(D107-A2): track 0.00 -> 2.95 mm
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