File: hardware/modules/IGNRocketOrderFile/Rocket/LiPoPower2.kicad_sch (KiCad schematic)
At the start: 49 parts, among them J401 Conn_01x03, J402 Ext Switch, J403 LiPo, U401 TPS2116DRL, U402 MCP73871-1CC, U403 INA226, U404 INA226, U405 TPS63070RNMR, U406 INA226

Commit message: 発注基板修正
Parts:
- R411: footprint Resistor_SMD:R_0402_1005Metric -> Resistor_SMD:R_0603_1608Metric
