File: hardware/modules/IGNRocketOrderFile/IGN/RP2040Core.kicad_sch (KiCad schematic)
At the start: 41 parts, among them J1301 DEBUG, SW1301 RESET_sw, SW1302 BOOT0, U1301 SN65HVD230, U1302 W25Q128JVS, U1303 RP2040, Y1301 Crystal_GND24

Commit message: 発注基板修正
Parts:
- renumbered C1301 to C301, C1302 to C302, C1303 to C303, C1304 to C304, C1305 to C305, C1306 to C306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
