File: hardware/modules/Tri.Ctrl1/Tri.Ctrl1.kicad_sch (KiCad schematic)
At the start: 5 parts, among them J101 ジョイコン1, J102 ジョイコン2, J103 トリム, J104 7セグ

Commit message: 主にCAN周りの修正
Parts:
- renumbered J104 to J103, J103 to J104
Connections:
- no-connect marks 7 -> 8
Other:
- sheet IF-MR ports: added none; removed EN
Changed lines of the file:
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@@
 		(at 92.075 123.825)
+	)
+	(no_connect
+		(at 92.075 78.105)
 	)
 	(bus_entry
@@
 	(wire
 		(pts
-			(xy 86.995 78.105) (xy 86.995 60.325)
-		)
-		(stroke
-			(width 0)
-			(type default)
-		)
-	)
-	(wire
-		(pts
 			(xy 68.58 113.665) (xy 29.845 113.665)
 		)
@@
 		)
 	)
-	(wire
-		(pts
-			(xy 92.075 78.105) (xy 86.995 78.105)
-		)
-		(stroke
-			(width 0)
-			(type default)
-		)
-	)
 	(bus
 		(pts
@@
 		)
 	)
-	(wire
-		(pts
-			(xy 86.995 60.325) (xy 164.465 60.325)
-		)
-		(stroke
-			(width 0)
-			(type default)
-		)
-	)
 	(bus
 		(pts
@@
 	(wire
 		(pts
-			(xy 164.465 60.325) (xy 164.465 67.945)
-		)
-		(stroke
-			(width 0)
-			(type default)
-		)
-	)
-	(wire
-		(pts
 			(xy 83.82 118.745) (xy 92.075 118.745)
 		)
@@
 		(pts
 			(xy 167.64 85.725) (xy 167.64 88.265)
-		)
-		(stroke
-			(width 0)
-			(type default)
-		)
-	)
-	(wire
-		(pts
-			(xy 164.465 67.945) (xy 197.485 67.945)
 		)
 		(stroke
@@
 		(dnp no)
 		(fields_autoplaced yes)
-		(property "Reference" "J103"
+		(property "Reference" "J104"
 			(at 144.145 146.05 0)
 			(effects
@@
 			(project ""
 				(path "/39a3f286-a766-4612-a8bf-4e53d682d5ae"
-					(reference "J103")
+					(reference "J104")
 					(unit 1)
 				)
@@
 		(dnp no)
 		(fields_autoplaced yes)
-		(property "Reference" "#PWR0106"
+		(property "Reference" "#PWR0109"
 			(at 151.13 161.925 0)
 			(effects
@@
 			(project ""
 				(path "/39a3f286-a766-4612-a8bf-4e53d682d5ae"
-					(reference "#PWR0106")
+					(reference "#PWR0109")
 					(unit 1)
 				)
@@
 		(dnp no)
 		(fields_autoplaced yes)
-		(property "Reference" "#PWR0108"
+		(property "Reference" "#PWR0106"
 			(at 56.515 160.655 0)
 			(effects
@@
 			(project ""
 				(path "/39a3f286-a766-4612-a8bf-4e53d682d5ae"
-					(reference "#PWR0108")
+					(reference "#PWR0106")
 					(unit 1)
 				)
@@
 		(dnp no)
 		(fields_autoplaced yes)
-		(property "Reference" "#PWR0105"
+		(property "Reference" "#PWR0107"
 			(at 74.93 72.39 0)
 			(effects
@@
 			(project "Tri.Ctrl1"
 				(path "/39a3f286-a766-4612-a8bf-4e53d682d5ae"
-					(reference "#PWR0105")
+					(reference "#PWR0107")
 					(unit 1)
 				)
@@
 		(dnp no)
 		(fields_autoplaced yes)
-		(property "Reference" "J104"
+		(property "Reference" "J103"
 			(at 43.18 146.685 0)
 			(effects
@@
 			(project ""
 				(path "/39a3f286-a766-4612-a8bf-4e53d682d5ae"
-					(reference "J104")
+					(reference "J103")
 					(unit 1)
 				)
@@
 		(dnp no)
 		(fields_autoplaced yes)
-		(property "Reference" "#PWR0109"
+		(property "Reference" "#PWR0108"
 			(at 90.17 71.12 0)
 			(effects
@@
 			(project ""
 				(path "/39a3f286-a766-4612-a8bf-4e53d682d5ae"
-					(reference "#PWR0109")
+					(reference "#PWR0108")
 					(unit 1)
 				)
@@
 		(dnp no)
 		(fields_autoplaced yes)
-		(property "Reference" "#PWR0107"
+		(property "Reference" "#PWR0105"
 			(at 56.515 155.575 0)
 			(effects
@@
 			(project ""
 				(path "/39a3f286-a766-4612-a8bf-4e53d682d5ae"
-					(reference "#PWR0107")
+					(reference "#PWR0105")
 					(unit 1)
 				)
@@
 			(effects
 				(font
-					(size 1.27 1.27)
-				)
-				(justify left)
-			)
-		)
-		(pin "EN" input
-			(at 197.485 67.945 180)
-			(effects
-				(font
