File: hardware/modules/Tri.MR/Pressure.kicad_sch (KiCad schematic)
At the start: 5 parts

Commit message: 回路図完成，部品配置完了，一部配線終了
Parts:
- U301: renamed from U101; footprint WOBClibrary:BME280 -> WOBCLibrary:BME280
- renumbered C101 to C301, C102 to C302, C103 to C303, C104 to C304
Changed lines of the file:
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@@
 		(on_board yes)
 		(dnp no)
-		(property "Reference" "C102"
+		(property "Reference" "C302"
 			(at 117.856 108.458 0)
 			(effects
@@
 			(project "Pressure"
 				(path "/09ffad5f-d798-427b-afb7-94e9cea30a78/fed7b5e5-0cf8-4f36-b77c-4bbd1eb1c12f"
-					(reference "C102")
+					(reference "C302")
 					(unit 1)
 				)
@@
 		(on_board yes)
 		(dnp no)
-		(property "Reference" "C101"
+		(property "Reference" "C301"
 			(at 109.982 108.204 0)
 			(effects
@@
 			(project "Pressure"
 				(path "/09ffad5f-d798-427b-afb7-94e9cea30a78/fed7b5e5-0cf8-4f36-b77c-4bbd1eb1c12f"
-					(reference "C101")
+					(reference "C301")
 					(unit 1)
 				)
@@
 		(on_board yes)
 		(dnp no)
-		(property "Reference" "C103"
+		(property "Reference" "C303"
 			(at 125.73 108.458 0)
 			(effects
@@
 			(project "Pressure"
 				(path "/09ffad5f-d798-427b-afb7-94e9cea30a78/fed7b5e5-0cf8-4f36-b77c-4bbd1eb1c12f"
-					(reference "C103")
+					(reference "C303")
 					(unit 1)
 				)
@@
 		(dnp no)
 		(fields_autoplaced yes)
-		(property "Reference" "U101"
+		(property "Reference" "U301"
 			(at 130.81 85.09 0)
 			(effects
@@
 			)
 		)
-		(property "Footprint" "WOBClibrary:BME280"
+		(property "Footprint" "WOBCLibrary:BME280"
 			(at 130.81 95.25 0)
 			(effects
@@
 			(project "Pressure"
 				(path "/09ffad5f-d798-427b-afb7-94e9cea30a78/fed7b5e5-0cf8-4f36-b77c-4bbd1eb1c12f"
-					(reference "U101")
+					(reference "U301")
 					(unit 1)
 				)
@@
 		(dnp no)
 		(fields_autoplaced yes)
-		(property "Reference" "#PWR0101"
+		(property "Reference" "#PWR0301"
 			(at 138.43 124.46 0)
 			(effects
@@
 			(project "Pressure"
 				(path "/09ffad5f-d798-427b-afb7-94e9cea30a78/fed7b5e5-0cf8-4f36-b77c-4bbd1eb1c12f"
-					(reference "#PWR0101")
+					(reference "#PWR0301")
 					(unit 1)
 				)
@@
 		(dnp no)
 		(fields_autoplaced yes)
-		(property "Reference" "#FLG0101"
+		(property "Reference" "#FLG0301"
 			(at 130.81 120.015 0)
 			(effects
@@
 			(project "Pressure"
 				(path "/09ffad5f-d798-427b-afb7-94e9cea30a78/fed7b5e5-0cf8-4f36-b77c-4bbd1eb1c12f"
-					(reference "#FLG0101")
+					(reference "#FLG0301")
 					(unit 1)
 				)
@@
 		(on_board yes)
 		(dnp no)
-		(property "Reference" "C104"
+		(property "Reference" "C304"
 			(at 135.128 108.204 0)
 			(effects
@@
 			(project "Pressure"
 				(path "/09ffad5f-d798-427b-afb7-94e9cea30a78/fed7b5e5-0cf8-4f36-b77c-4bbd1eb1c12f"
-					(reference "C104")
-					(unit 1)
-				)
+					(reference "C304")
+					(unit 1)
+				)
