File: hardware/modules/Tri.Ctrl2/ESP32Core.kicad_sch (KiCad schematic)
At the start: 22 parts, among them SW1 RESET_sw, U1 TPS3820, U2 SN65HVD230, U3 ESP32-S3-WROOM-1

Commit message: 回路図ひととおり完了
Parts:
- added R201: 10k, Resistor_SMD:R_0402_1005Metric, symbol Device:R
Connections:
- net VDD: now also R201.1
- net at SW1.1, U1.3 (MR): now also R201.2
Other:
- moved on the sheet: SW1

Commit message: ひととおり配置
Parts:
- U1: footprint PCM_Package_TO_SOT_SMD_AKL:SOT-23-5 -> Package_TO_SOT_SMD:SOT-23-5
Changed lines of the file:
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@@
 			)
 		)
-		(property "Footprint" "PCM_Package_TO_SOT_SMD_AKL:SOT-23-5"
+		(property "Footprint" "Package_TO_SOT_SMD:SOT-23-5"
 			(at 40.005 104.775 0)
 			(effects

Commit message: LCSC最終確認
Parts:
- R201: LCSC C25117 -> C25744
Changed lines of the file:
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@@
 			)
 		)
-		(property "LCSC" "C25117"
+		(property "LCSC" "C25744"
 			(at 53.34 98.425 0)
 			(effects

Commit message: 新しいバージョンで保存
Parts:
- renumbered C1 to C201, C2 to C202, C3 to C203, C4 to C204, D1 to D201, D2 to D202, D3 to D203, D4 to D204, D5 to D205, D6 to D206, R1 to R202, R2 to R203, R3 to R204, R4 to R205, R5 to R206, R6 to R207, R7 to R208, SW1 to SW201, U1 to U201, U2 to U202, U3 to U203, USB1 to USB201
