File: hardware/modules/IGN/Pressure.kicad_sch (KiCad schematic)
At the start: 5 parts

Commit message: 回路図は一旦終了
Parts:
- U501: renamed from U101; footprint WOBClibrary:BME280 -> WOBCLibrary:BME280
- renumbered C101 to C501, C102 to C502, C103 to C503, C104 to C504
Changed lines of the file:
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@@
 		(on_board yes)
 		(dnp no)
-		(property "Reference" "C102"
+		(property "Reference" "C502"
 			(at 117.856 108.458 0)
 			(effects
@@
 			(project "Pressure"
 				(path "/2a7771e6-36a4-47ae-b559-dde705e1d286/3c4b5ceb-c9aa-4ec9-ae4e-83d5decb932e"
-					(reference "C102")
+					(reference "C502")
 					(unit 1)
 				)
@@
 		(on_board yes)
 		(dnp no)
-		(property "Reference" "C101"
+		(property "Reference" "C501"
 			(at 109.982 108.204 0)
 			(effects
@@
 			(project "Pressure"
 				(path "/2a7771e6-36a4-47ae-b559-dde705e1d286/3c4b5ceb-c9aa-4ec9-ae4e-83d5decb932e"
-					(reference "C101")
+					(reference "C501")
 					(unit 1)
 				)
@@
 		(on_board yes)
 		(dnp no)
-		(property "Reference" "C103"
+		(property "Reference" "C503"
 			(at 125.73 108.458 0)
 			(effects
@@
 			(project "Pressure"
 				(path "/2a7771e6-36a4-47ae-b559-dde705e1d286/3c4b5ceb-c9aa-4ec9-ae4e-83d5decb932e"
-					(reference "C103")
+					(reference "C503")
 					(unit 1)
 				)
@@
 		(dnp no)
 		(fields_autoplaced yes)
-		(property "Reference" "U101"
+		(property "Reference" "U501"
 			(at 130.81 85.09 0)
 			(effects
@@
 			)
 		)
-		(property "Footprint" "WOBClibrary:BME280"
+		(property "Footprint" "WOBCLibrary:BME280"
 			(at 130.81 95.25 0)
 			(effects
@@
 			(project "Pressure"
 				(path "/2a7771e6-36a4-47ae-b559-dde705e1d286/3c4b5ceb-c9aa-4ec9-ae4e-83d5decb932e"
-					(reference "U101")
+					(reference "U501")
 					(unit 1)
 				)
@@
 		(dnp no)
 		(fields_autoplaced yes)
-		(property "Reference" "#PWR0101"
+		(property "Reference" "#PWR0501"
 			(at 138.43 124.46 0)
 			(effects
@@
 			(project "Pressure"
 				(path "/2a7771e6-36a4-47ae-b559-dde705e1d286/3c4b5ceb-c9aa-4ec9-ae4e-83d5decb932e"
-					(reference "#PWR0101")
+					(reference "#PWR0501")
 					(unit 1)
 				)
@@
 		(dnp no)
 		(fields_autoplaced yes)
-		(property "Reference" "#FLG0101"
+		(property "Reference" "#FLG0501"
 			(at 130.81 120.015 0)
 			(effects
@@
 			(project "Pressure"
 				(path "/2a7771e6-36a4-47ae-b559-dde705e1d286/3c4b5ceb-c9aa-4ec9-ae4e-83d5decb932e"
-					(reference "#FLG0101")
+					(reference "#FLG0501")
 					(unit 1)
 				)
@@
 		(on_board yes)
 		(dnp no)
-		(property "Reference" "C104"
+		(property "Reference" "C504"
 			(at 135.128 108.204 0)
 			(effects
@@
 			(project "Pressure"
 				(path "/2a7771e6-36a4-47ae-b559-dde705e1d286/3c4b5ceb-c9aa-4ec9-ae4e-83d5decb932e"
-					(reference "C104")
-					(unit 1)
-				)
+					(reference "C504")
+					(unit 1)
+				)
