File: hardware/modules/RCS/LoadCell2.kicad_sch (KiCad schematic)
At the start: 12 parts, among them J101 Conn_01x04, Q101 PNP, U101 HX711

Commit message: RCS回路作成
Parts:
- removed C101, C104: 10uF, Capacitor_SMD:C_0603_1608Metric, symbol Device:C
- removed C102, C103, C105: 0.1uF, Capacitor_SMD:C_0402_1005Metric, symbol Device:C
- removed J101: Conn_01x04, Connector_JST:JST_PH_B4B-PH-K_1x04_P2.00mm_Vertical, symbol Connector_Generic:Conn_01x04
- removed Q101: PNP, Package_TO_SOT_SMD:SOT-23, symbol Simulation_SPICE:PNP
- removed R101, R102: 100, Resistor_SMD:R_0402_1005Metric, symbol Device:R
- removed R103: 22k, Resistor_SMD:R_0402_1005Metric, symbol Device:R
- removed R104: 10k, Resistor_SMD:R_0402_1005Metric, symbol Device:R
- removed U101: HX711, Package_SO:SOP-16_3.9x9.9mm_P1.27mm, symbol Analog_ADC:HX711
- added C131, C134: 10uF, Capacitor_SMD:C_0603_1608Metric, symbol Device:C
- added C132, C133, C135: 0.1uF, Capacitor_SMD:C_0402_1005Metric, symbol Device:C
- added J108: Conn_01x04, Connector_JST:JST_PH_B4B-PH-K_1x04_P2.00mm_Vertical, symbol Connector_Generic:Conn_01x04
- added Q104: PNP, Package_TO_SOT_SMD:SOT-23, symbol Simulation_SPICE:PNP
- added R124, R125: 100, Resistor_SMD:R_0402_1005Metric, symbol Device:R
- added R126: 22k, Resistor_SMD:R_0402_1005Metric, symbol Device:R
- added R127: 10k, Resistor_SMD:R_0402_1005Metric, symbol Device:R
- added U107: HX711, Package_SO:SOP-16_3.9x9.9mm_P1.27mm, symbol Analog_ADC:HX711
Connections:
- net CLK: now also U107.11 (PD_SCK)
- net DAT: now also U107.12 (DOUT)
- net GND: now also C131.2, C133.2, C134.2, C135.2, J108.3 (Pin_3), R127.2, U107.10 (INB+), U107.14 (XI), U107.5 (AGND), U107.9 (INB-)
- net VDD: now also C134.1, C135.1, Q104.3 (E), R126.1, U107.1 (VSUP), U107.15 (RATE), U107.16 (DVDD), U107.3 (AVDD)
- new net: Q104.2 (B), U107.2 (BASE)
- new net: R126.2, R127.1, U107.4 (VFB)
- new net: C133.1, U107.6 (VBG)
- new net: C132.2, R125.2, U107.7 (INA-)
- new net: C132.1, R124.2, U107.8 (INA+)
- new net: J108.2 (Pin_2), R125.1
- new net: C131.1, J108.4 (Pin_4), Q104.1 (C)
- new net: J108.1 (Pin_1), R124.1

Commit message: loadcell消してIMUとPressure追加
Parts:
- renumbered C131 to C601, C132 to C602, C133 to C603, C134 to C604, C135 to C605, J108 to J601, Q104 to Q601, R124 to R601, R125 to R602, R126 to R603, R127 to R604, U107 to U601
Changed lines of the file:
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@@
 (kicad_sch
-	(version 20231120)
+	(version 20250114)
 	(generator "eeschema")
-	(generator_version "8.0")
+	(generator_version "9.0")
 	(paper "A4")
 	(junction
@@
 		(shape input)
 		(at 185.674 93.98 0)
-		(fields_autoplaced yes)
 		(effects
 			(font
@@
 		(shape input)
 		(at 185.674 96.52 0)
-		(fields_autoplaced yes)
 		(effects
 			(font
@@
 		(on_board yes)
 		(dnp no)
-		(property "Reference" "#PWR0159"
+		(property "Reference" "#PWR0607"
 			(at 183.134 125.73 0)
 			(effects
@@
 			(project "RCS"
 				(path "/8712227c-dfcf-4399-a04c-a9abd63db3ea/db154cb7-eab6-448f-a7fe-5bcfbe31da61"
-					(reference "#PWR0159")
+					(reference "#PWR0607")
 					(unit 1)
 				)
@@
 		(dnp no)
 		(fields_autoplaced yes)
-		(property "Reference" "C134"
+		(property "Reference" "C604"
 			(at 156.718 73.9139 0)
 			(effects
@@
 			(project "RCS"
 				(path "/8712227c-dfcf-4399-a04c-a9abd63db3ea/db154cb7-eab6-448f-a7fe-5bcfbe31da61"
-					(reference "C134")
+					(reference "C604")
 					(unit 1)
 				)
@@
 		(dnp no)
 		(fields_autoplaced yes)
-		(property "Reference" "U107"
+		(property "Reference" "U601"
 			(at 169.5801 121.158 0)
 			(effects
@@
 			(project "RCS"
 				(path "/8712227c-dfcf-4399-a04c-a9abd63db3ea/db154cb7-eab6-448f-a7fe-5bcfbe31da61"
-					(reference "U107")
+					(reference "U601")
 					(unit 1)
 				)
@@
 		(on_board yes)
 		(dnp no)
-		(property "Reference" "R125"
+		(property "Reference" "R602"
 			(at 128.778 112.268 90)
 			(effects
@@
 			(project "RCS"
 				(path "/8712227c-dfcf-4399-a04c-a9abd63db3ea/db154cb7-eab6-448f-a7fe-5bcfbe31da61"
-					(reference "R125")
+					(reference "R602")
 					(unit 1)
 				)
@@
 		(on_board yes)
 		(dnp no)
-		(property "Reference" "#PWR0158"
+		(property "Reference" "#PWR0606"
 			(at 183.134 113.792 0)
 			(effects
@@
 			(project "RCS"
 				(path "/8712227c-dfcf-4399-a04c-a9abd63db3ea/db154cb7-eab6-448f-a7fe-5bcfbe31da61"
-					(reference "#PWR0158")
+					(reference "#PWR0606")
 					(unit 1)
 				)
@@
 		(dnp no)
 		(fields_autoplaced yes)
-		(property "Reference" "#PWR0154"
+		(property "Reference" "#PWR0602"
 			(at 129.032 71.628 0)
 			(effects
@@
 			(project "RCS"
 				(path "/8712227c-dfcf-4399-a04c-a9abd63db3ea/db154cb7-eab6-448f-a7fe-5bcfbe31da61"
-					(reference "#PWR0154")
+					(reference "#PWR0602")
 					(unit 1)
 				)
@@
 		(dnp no)
 		(fields_autoplaced yes)
-		(property "Reference" "Q104"
+		(property "Reference" "Q601"
 			(at 126.238 83.5659 0)
 			(effects
@@
 			(project "RCS"
 				(path "/8712227c-dfcf-4399-a04c-a9abd63db3ea/db154cb7-eab6-448f-a7fe-5bcfbe31da61"
-					(reference "Q104")
+					(reference "Q601")
 					(unit 1)
 				)
@@
 		(on_board yes)
 		(dnp no)
-		(property "Reference" "#PWR0155"
+		(property "Reference" "#PWR0603"
 			(at 141.986 108.966 0)
 			(effects
@@
 			(project "RCS"
 				(path "/8712227c-dfcf-4399-a04c-a9abd63db3ea/db154cb7-eab6-448f-a7fe-5bcfbe31da61"
-					(reference "#PWR0155")
+					(reference "#PWR0603")
 					(unit 1)
 				)
@@
 		(on_board yes)
 		(dnp no)
-		(property "Reference" "J108"
+		(property "Reference" "J601"
 			(at 114.808 96.774 0)
 			(effects
@@
 			(project "RCS"
 				(path "/8712227c-dfcf-4399-a04c-a9abd63db3ea/db154cb7-eab6-448f-a7fe-5bcfbe31da61"
-					(reference "J108")
+					(reference "J601")
 					(unit 1)
 				)
@@
 		(on_board yes)
 		(dnp no)
-		(property "Reference" "C132"
+		(property "Reference" "C602"
 			(at 137.922 117.094 0)
 			(effects
@@
 			(project "RCS"
 				(path "/8712227c-dfcf-4399-a04c-a9abd63db3ea/db154cb7-eab6-448f-a7fe-5bcfbe31da61"
-					(reference "C132")
+					(reference "C602")
 					(unit 1)
 				)
@@
 		(on_board yes)
 		(dnp no)
-		(property "Reference" "C135"
+		(property "Reference" "C605"
 			(at 183.896 113.284 0)
 			(effects
@@
 			(project "RCS"
 				(path "/8712227c-dfcf-4399-a04c-a9abd63db3ea/db154cb7-eab6-448f-a7fe-5bcfbe31da61"
-					(reference "C135")
+					(reference "C605")
 					(unit 1)
 				)
@@
 		(on_board yes)
 		(dnp no)
-		(property "Reference" "C131"
+		(property "Reference" "C601"
 			(at 125.984 98.044 0)
 			(effects
@@
 			(project "RCS"
 				(path "/8712227c-dfcf-4399-a04c-a9abd63db3ea/db154cb7-eab6-448f-a7fe-5bcfbe31da61"
-					(reference "C131")
+					(reference "C601")
 					(unit 1)
 				)
@@
 		(dnp no)
 		(fields_autoplaced yes)
-		(property "Reference" "#PWR0153"
+		(property "Reference" "#PWR0601"
 			(at 123.19 122.428 0)
 			(effects
@@
 			(project "RCS"
 				(path "/8712227c-dfcf-4399-a04c-a9abd63db3ea/db154cb7-eab6-448f-a7fe-5bcfbe31da61"
-					(reference "#PWR0153")
+					(reference "#PWR0601")
 					(unit 1)
 				)
@@
 		(dnp no)
 		(fields_autoplaced yes)
-		(property "Reference" "#PWR0157"
+		(property "Reference" "#PWR0605"
 			(at 167.386 131.826 0)
 			(effects
@@
 			(project "RCS"
 				(path "/8712227c-dfcf-4399-a04c-a9abd63db3ea/db154cb7-eab6-448f-a7fe-5bcfbe31da61"
-					(reference "#PWR0157")
+					(reference "#PWR0605")
 					(unit 1)
 				)
@@
 		(on_board yes)
 		(dnp no)
-		(property "Reference" "C133"
+		(property "Reference" "C603"
 			(at 153.416 118.364 0)
 			(effects
@@
 			(project "RCS"
 				(path "/8712227c-dfcf-4399-a04c-a9abd63db3ea/db154cb7-eab6-448f-a7fe-5bcfbe31da61"
-					(reference "C133")
+					(reference "C603")
 					(unit 1)
 				)
@@
 		(on_board yes)
 		(dnp no)
-		(property "Reference" "R126"
+		(property "Reference" "R603"
 			(at 143.51 79.248 0)
 			(effects
@@
 			(project "RCS"
 				(path "/8712227c-dfcf-4399-a04c-a9abd63db3ea/db154cb7-eab6-448f-a7fe-5bcfbe31da61"
-					(reference "R126")
+					(reference "R603")
 					(unit 1)
 				)
@@
 		(dnp no)
 		(fields_autoplaced yes)
-		(property "Reference" "#PWR0156"
+		(property "Reference" "#PWR0604"
 			(at 153.162 85.344 0)
 			(effects
@@
 			(project "RCS"
 				(path "/8712227c-dfcf-4399-a04c-a9abd63db3ea/db154cb7-eab6-448f-a7fe-5bcfbe31da61"
-					(reference "#PWR0156")
+					(reference "#PWR0604")
 					(unit 1)
 				)
@@
 		(on_board yes)
 		(dnp no)
-		(property "Reference" "#PWR0160"
+		(property "Reference" "#PWR0608"
 			(at 186.69 111.76 0)
 			(effects
@@
 			(project "RCS"
 				(path "/8712227c-dfcf-4399-a04c-a9abd63db3ea/db154cb7-eab6-448f-a7fe-5bcfbe31da61"
-					(reference "#PWR0160")
+					(reference "#PWR0608")
 					(unit 1)
 				)
@@
 		(on_board yes)
 		(dnp no)
-		(property "Reference" "R124"
+		(property "Reference" "R601"
 			(at 128.27 105.156 90)
 			(effects
@@
 			(project "RCS"
 				(path "/8712227c-dfcf-4399-a04c-a9abd63db3ea/db154cb7-eab6-448f-a7fe-5bcfbe31da61"
-					(reference "R124")
+					(reference "R601")
 					(unit 1)
 				)
@@
 		(on_board yes)
 		(dnp no)
-		(property "Reference" "R127"
+		(property "Reference" "R604"
 			(at 143.51 96.774 0)
 			(effects
@@
 			(project "RCS"
 				(path "/8712227c-dfcf-4399-a04c-a9abd63db3ea/db154cb7-eab6-448f-a7fe-5bcfbe31da61"
-					(reference "R127")
+					(reference "R604")
 					(unit 1)
 				)
