File: hardware/modules/MissionBus/IMU2.kicad_sch (KiCad schematic)
At the start: 10 parts, among them U1001 BMM150, U1002 BMI270

Commit message: LCSC確認後，再度ガーバーファイル出力
Parts:
- C1001, C1003, C1005, C1007: LCSC (none) -> C19702
- C1002, C1004, C1006, C1008: LCSC (none) -> C1525
Changed lines of the file:
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@@
+			)
+		)
+		(property "LCSC" "C1525"
+			(at 130.81 83.82 0)
+			(effects
+				(font
+					(size 1.27 1.27)
+				)
+				(hide yes)
 			)
 		)
@@
 			)
 		)
+		(property "LCSC" "C19702"
+			(at 125.73 83.82 0)
+			(effects
+				(font
+					(size 1.27 1.27)
+				)
+				(hide yes)
+			)
+		)
 		(pin "2"
 		)
@@
 		)
 		(property "Description" "Unpolarized capacitor"
+			(at 118.11 101.6 0)
+			(effects
+				(font
+					(size 1.27 1.27)
+				)
+				(hide yes)
+			)
+		)
+		(property "LCSC" "C19702"
 			(at 118.11 101.6 0)
 			(effects
@@
 			)
 		)
+		(property "LCSC" "C1525"
+			(at 238.76 109.22 0)
+			(effects
+				(font
+					(size 1.27 1.27)
+				)
+				(hide yes)
+			)
+		)
 		(pin "2"
 		)
@@
 		)
 		(property "Description" "Unpolarized capacitor"
+			(at 232.41 109.22 0)
+			(effects
+				(font
+					(size 1.27 1.27)
+				)
+				(hide yes)
+			)
+		)
+		(property "LCSC" "C19702"
 			(at 232.41 109.22 0)
 			(effects
@@
 			)
 		)
+		(property "LCSC" "C1525"
+			(at 123.19 101.6 0)
+			(effects
+				(font
+					(size 1.27 1.27)
+				)
+				(hide yes)
+			)
+		)
 		(pin "1"
 		)
@@
 			)
 		)
+		(property "LCSC" "C1525"
+			(at 218.44 106.68 0)
+			(effects
+				(font
+					(size 1.27 1.27)
+				)
+				(hide yes)
+			)
+		)
 		(pin "1"
 		)
@@
 			(at 212.09 106.68 0)
 			(effects
+				(font
+					(size 1.27 1.27)
+				)
+				(hide yes)
+			)
+		)
+		(property "LCSC" "C19702"
+			(at 212.09 106.68 0)
+			(effects
