File: hardware/modules/Rocket_ver_G/LoRa.kicad_sch (KiCad schematic)
At the start: 13 parts, among them J101 SMA, J102 SMA, U101 E220-900T22S(JP)

Commit message: 途中経過
Changed lines of the file:
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@@
 (kicad_sch
-	(version 20231120)
+	(version 20250114)
 	(generator "eeschema")
-	(generator_version "8.0")
+	(generator_version "9.0")
 	(paper "A4")
 	(junction
@@
 		(shape output)
 		(at 194.31 102.87 0)
-		(fields_autoplaced yes)
 		(effects
 			(font
@@
 		(shape output)
 		(at 194.31 92.71 0)
-		(fields_autoplaced yes)
 		(effects
 			(font
@@
 		(shape input)
 		(at 135.89 102.87 0)
-		(fields_autoplaced yes)
 		(effects
 			(font
@@
 		(shape output)
 		(at 194.31 100.33 0)
-		(fields_autoplaced yes)
 		(effects
 			(font
@@
 		(shape output)
 		(at 194.31 95.25 0)
-		(fields_autoplaced yes)
 		(effects
 			(font
@@
 		(shape input)
 		(at 194.31 97.79 0)
-		(fields_autoplaced yes)
 		(effects
 			(font
@@
 		(shape input)
 		(at 135.89 97.79 0)
-		(fields_autoplaced yes)
 		(effects
 			(font
@@
 		(instances
 			(project "LoRa"
+				(path "/718e9fc1-0aec-4051-b929-e6ccf2afef13/62d39229-64df-434c-b537-8e099071c95b"
+					(reference "#PWR0101")
+					(unit 1)
+				)
+			)
+			(project "LoRa"
 				(path "/d339b9d8-51a7-460e-bb19-8d8c25d3e2aa"
 					(reference "#PWR0101")
@@
 		)
 		(instances
+			(project "LoRa"
+				(path "/718e9fc1-0aec-4051-b929-e6ccf2afef13/62d39229-64df-434c-b537-8e099071c95b"
+					(reference "C107")
+					(unit 1)
+				)
+			)
 			(project "LoRa"
 				(path "/d339b9d8-51a7-460e-bb19-8d8c25d3e2aa"
@@
 		(instances
 			(project "LoRa"
+				(path "/718e9fc1-0aec-4051-b929-e6ccf2afef13/62d39229-64df-434c-b537-8e099071c95b"
+					(reference "D102")
+					(unit 1)
+				)
+			)
+			(project "LoRa"
 				(path "/d339b9d8-51a7-460e-bb19-8d8c25d3e2aa"
 					(reference "D102")
@@
 		(instances
 			(project "LoRa"
+				(path "/718e9fc1-0aec-4051-b929-e6ccf2afef13/62d39229-64df-434c-b537-8e099071c95b"
+					(reference "Switch101")
+					(unit 1)
+				)
+			)
+			(project "LoRa"
 				(path "/d339b9d8-51a7-460e-bb19-8d8c25d3e2aa"
 					(reference "Switch101")
@@
 		(instances
 			(project "LoRa"
+				(path "/718e9fc1-0aec-4051-b929-e6ccf2afef13/62d39229-64df-434c-b537-8e099071c95b"
+					(reference "C103")
+					(unit 1)
+				)
+			)
+			(project "LoRa"
 				(path "/d339b9d8-51a7-460e-bb19-8d8c25d3e2aa"
 					(reference "C103")
@@
 		(instances
 			(project "LoRa"
+				(path "/718e9fc1-0aec-4051-b929-e6ccf2afef13/62d39229-64df-434c-b537-8e099071c95b"
+					(reference "C102")
+					(unit 1)
+				)
+			)
+			(project "LoRa"
 				(path "/d339b9d8-51a7-460e-bb19-8d8c25d3e2aa"
 					(reference "C102")
@@
 		)
 		(instances
+			(project "LoRa"
+				(path "/718e9fc1-0aec-4051-b929-e6ccf2afef13/62d39229-64df-434c-b537-8e099071c95b"
+					(reference "C104")
+					(unit 1)
+				)
+			)
 			(project "LoRa"
 				(path "/d339b9d8-51a7-460e-bb19-8d8c25d3e2aa"
@@
 		(instances
 			(project "LoRa"
+				(path "/718e9fc1-0aec-4051-b929-e6ccf2afef13/62d39229-64df-434c-b537-8e099071c95b"
+					(reference "J102")
+					(unit 1)
+				)
+			)
+			(project "LoRa"
 				(path "/d339b9d8-51a7-460e-bb19-8d8c25d3e2aa"
 					(reference "J102")
@@
 		(instances
 			(project "LoRa"
+				(path "/718e9fc1-0aec-4051-b929-e6ccf2afef13/62d39229-64df-434c-b537-8e099071c95b"
+					(reference "C101")
+					(unit 1)
+				)
+			)
+			(project "LoRa"
 				(path "/d339b9d8-51a7-460e-bb19-8d8c25d3e2aa"
 					(reference "C101")
@@
 		)
 		(instances
+			(project "LoRa"
+				(path "/718e9fc1-0aec-4051-b929-e6ccf2afef13/62d39229-64df-434c-b537-8e099071c95b"
+					(reference "D101")
+					(unit 1)
+				)
+			)
 			(project "LoRa"
 				(path "/d339b9d8-51a7-460e-bb19-8d8c25d3e2aa"
@@
 		(instances
 			(project "LoRa"
+				(path "/718e9fc1-0aec-4051-b929-e6ccf2afef13/62d39229-64df-434c-b537-8e099071c95b"
+					(reference "J101")
+					(unit 1)
+				)
+			)
+			(project "LoRa"
 				(path "/d339b9d8-51a7-460e-bb19-8d8c25d3e2aa"
 					(reference "J101")
@@
 		)
 		(instances
+			(project "LoRa"
+				(path "/718e9fc1-0aec-4051-b929-e6ccf2afef13/62d39229-64df-434c-b537-8e099071c95b"
+					(reference "C105")
+					(unit 1)
+				)
+			)
 			(project "LoRa"
 				(path "/d339b9d8-51a7-460e-bb19-8d8c25d3e2aa"
@@
 		(instances
 			(project "LoRa"
+				(path "/718e9fc1-0aec-4051-b929-e6ccf2afef13/62d39229-64df-434c-b537-8e099071c95b"
+					(reference "U101")
+					(unit 1)
+				)
+			)
+			(project "LoRa"
 				(path "/d339b9d8-51a7-460e-bb19-8d8c25d3e2aa"
 					(reference "U101")
@@
 		(instances
 			(project "LoRa"
+				(path "/718e9fc1-0aec-4051-b929-e6ccf2afef13/62d39229-64df-434c-b537-8e099071c95b"
+					(reference "C106")
+					(unit 1)
+				)
+			)
+			(project "LoRa"
 				(path "/d339b9d8-51a7-460e-bb19-8d8c25d3e2aa"
 					(reference "C106")
@@
 		)
 	)
-	(sheet_instances
-		(path "/"
-			(page "1")
-		)
-	)

Commit message: 回路図まで
Parts:
- removed C101, C102, C105: 100p, Capacitor_SMD:C_0603_1608Metric, symbol Device:C_Small
- removed C103, C104: 100n, Capacitor_SMD:C_0402_1005Metric, symbol Device:C_Small
- removed D101, D102: ESD9B5.0ST5G, Diode_SMD:D_SOD-882, symbol Diode:ESD9B5.0ST5G
- removed J101, J102: SMA, Connector_Coaxial:SMA_Amphenol_132203-12_Horizontal, symbol Connector:Conn_Coaxial_Power
- removed Switch101: XA17-G4K1, Package_TO_SOT_SMD:SOT-363_SC-70-6, symbol XA17-G4K:XA17-G4K
- renumbered C106 to C701, C107 to C702, U101 to U701
