File: hardware/components/MotorControl/MotorControl.kicad_sch (KiCad schematic)
At the start: 12 parts, among them J1 MotorDriver, J2 ch1, J3 ch2, U1 LM2903PWR

Commit message: 回転数計コンポーネントなど
Parts:
- added R101, R102, R103, R104: 100, symbol Device:R
Connections:
- net IN1: now also R101.1; no longer J1.1 (Pin_1)
- net IN2: now also R102.1; no longer J1.2 (Pin_2)
- net IN3: now also R103.1; no longer J1.3 (Pin_3)
- net IN4: now also R104.1; no longer J1.4 (Pin_4)
- new net: J1.2 (Pin_2), R102.2
- new net: J1.1 (Pin_1), R101.2
- new net: J1.3 (Pin_3), R103.2
- new net: J1.4 (Pin_4), R104.2
