File: hardware/modules/CMG/CMGSon/ModuleIFSimple1.kicad_sch (KiCad schematic)
At the start: 4 parts, among them J401 Jumper, J402 Conn_01x04_MountingPin

Commit message: 一旦回路図完成
Parts:
- removed C401: 100nF, Capacitor_SMD:C_0402_1005Metric, symbol Device:C
- removed J401: Jumper, Connector_PinHeader_1.27mm:PinHeader_1x02_P1.27mm_Vertical, symbol Connector:Conn_01x02_Pin
- removed J402: Conn_01x04_MountingPin, WOBCLibrary:Grove_4P_L_SMD, symbol Connector_Generic_MountingPin:Conn_01x04_MountingPin
- removed R401: 120, Resistor_SMD:R_0402_1005Metric, symbol Device:R
- added C601: 100nF, Capacitor_SMD:C_0402_1005Metric, symbol Device:C
- added J601: Jumper, Connector_PinHeader_1.27mm:PinHeader_1x02_P1.27mm_Vertical, symbol Connector:Conn_01x02_Pin
- added J602: Conn_01x04_MountingPin, WOBCLibrary:Grove_4P_L_SMD, symbol Connector_Generic_MountingPin:Conn_01x04_MountingPin
- added R601: 120, Resistor_SMD:R_0402_1005Metric, symbol Device:R
Connections:
- net CANH: now also J602.1 (Pin_1), R601.2
- net CANL: now also J601.2 (Pin_2), J602.2 (Pin_2)
- net GND: now also C601.1, J602.4 (Pin_4), J602.MP (MountPin)
- net VIO: now also C601.2, J602.3 (Pin_3)
- new net: J601.1 (Pin_1), R601.1
