File: hardware/modules/CMG/CMGSon/Logger.kicad_sch (KiCad schematic)
At the start: 6 parts, among them U601 PCF8563T, Y601 Crystal

Commit message: コンポーネントを配置 サーボコンポーネントを追加
Parts:
- renumbered C602 to C20, C601 to C21, MICRO_SD601 to MICRO_SD1, U601 to U8, Y601 to Y1
Changed lines of the file:
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@@
 		(on_board yes)
 		(dnp no)
-		(property "Reference" "C602"
+		(property "Reference" "C20"
 			(at 140.97 85.725 0)
 			(effects
@@
 		)
 		(instances
+			(project "GS"
+				(path "/4eb245a9-6c21-4f00-ae42-6a498711dd85/fd7daa6e-d3a6-4f28-bda8-c91b24a77464"
+					(reference "C20")
+					(unit 1)
+				)
+			)
 			(project "GS"
 				(path "/920f9ee9-d8de-4f24-ad72-1c45434a67fe/2c35cf26-1e44-42e5-8139-efbe5f54c1ed"
@@
 		(instances
 			(project "CMGFather"
+				(path "/4eb245a9-6c21-4f00-ae42-6a498711dd85/fd7daa6e-d3a6-4f28-bda8-c91b24a77464"
+					(reference "#PWR0606")
+					(unit 1)
+				)
+			)
+			(project "CMGFather"
 				(path "/9e354a01-2cea-4232-8b65-4471166b2c2b/7ef76fdd-30f3-4139-a072-8ee3fa540a64"
 					(reference "#PWR0606")
@@
 		(dnp no)
 		(fields_autoplaced yes)
-		(property "Reference" "MICRO_SD601"
+		(property "Reference" "MICRO_SD1"
 			(at 117.475 76.2 0)
 			(effects
@@
 		)
 		(instances
+			(project "GS"
+				(path "/4eb245a9-6c21-4f00-ae42-6a498711dd85/fd7daa6e-d3a6-4f28-bda8-c91b24a77464"
+					(reference "MICRO_SD1")
+					(unit 1)
+				)
+			)
 			(project "GS"
 				(path "/920f9ee9-d8de-4f24-ad72-1c45434a67fe/2c35cf26-1e44-42e5-8139-efbe5f54c1ed"
@@
 		(on_board yes)
 		(dnp no)
-		(property "Reference" "#PWR0602"
+		(property "Reference" "#PWR063"
 			(at 185.42 84.455 0)
 			(effects
@@
 		)
 		(instances
+			(project "GS"
+				(path "/4eb245a9-6c21-4f00-ae42-6a498711dd85/fd7daa6e-d3a6-4f28-bda8-c91b24a77464"
+					(reference "#PWR063")
+					(unit 1)
+				)
+			)
 			(project "GS"
 				(path "/920f9ee9-d8de-4f24-ad72-1c45434a67fe/2c35cf26-1e44-42e5-8139-efbe5f54c1ed"
@@
 		(dnp no)
 		(fields_autoplaced yes)
-		(property "Reference" "#PWR0605"
+		(property "Reference" "#PWR065"
 			(at 190.5 107.315 0)
 			(effects
@@
 		)
 		(instances
+			(project "GS"
+				(path "/4eb245a9-6c21-4f00-ae42-6a498711dd85/fd7daa6e-d3a6-4f28-bda8-c91b24a77464"
+					(reference "#PWR065")
+					(unit 1)
+				)
+			)
 			(project "GS"
 				(path "/920f9ee9-d8de-4f24-ad72-1c45434a67fe/2c35cf26-1e44-42e5-8139-efbe5f54c1ed"
@@
 		(dnp no)
 		(fields_autoplaced yes)
-		(property "Reference" "#PWR0603"
+		(property "Reference" "#PWR061"
 			(at 145.415 86.36 0)
 			(effects
@@
 		)
 		(instances
+			(project "GS"
+				(path "/4eb245a9-6c21-4f00-ae42-6a498711dd85/fd7daa6e-d3a6-4f28-bda8-c91b24a77464"
+					(reference "#PWR061")
+					(unit 1)
+				)
+			)
 			(project "GS"
 				(path "/920f9ee9-d8de-4f24-ad72-1c45434a67fe/2c35cf26-1e44-42e5-8139-efbe5f54c1ed"
@@
 		(instances
 			(project "CMGFather"
+				(path "/4eb245a9-6c21-4f00-ae42-6a498711dd85/fd7daa6e-d3a6-4f28-bda8-c91b24a77464"
+					(reference "BT101")
+					(unit 1)
+				)
+			)
+			(project "CMGFather"
 				(path "/9e354a01-2cea-4232-8b65-4471166b2c2b/7ef76fdd-30f3-4139-a072-8ee3fa540a64"
 					(reference "BT101")
@@
 		(dnp no)
 		(fields_autoplaced yes)
-		(property "Reference" "U601"
+		(property "Reference" "U8"
 			(at 192.6941 78.105 0)
 			(effects
@@
 		)
 		(instances
+			(project "GS"
+				(path "/4eb245a9-6c21-4f00-ae42-6a498711dd85/fd7daa6e-d3a6-4f28-bda8-c91b24a77464"
+					(reference "U8")
+					(unit 1)
+				)
+			)
 			(project "GS"
 				(path "/920f9ee9-d8de-4f24-ad72-1c45434a67fe/2c35cf26-1e44-42e5-8139-efbe5f54c1ed"
@@
 		(dnp no)
 		(fields_autoplaced yes)
-		(property "Reference" "#PWR0604"
+		(property "Reference" "#PWR062"
 			(at 145.415 106.68 0)
 			(effects
@@
 		)
 		(instances
+			(project "GS"
+				(path "/4eb245a9-6c21-4f00-ae42-6a498711dd85/fd7daa6e-d3a6-4f28-bda8-c91b24a77464"
+					(reference "#PWR062")
+					(unit 1)
+				)
+			)
 			(project "GS"
 				(path "/920f9ee9-d8de-4f24-ad72-1c45434a67fe/2c35cf26-1e44-42e5-8139-efbe5f54c1ed"
@@
 		(on_board yes)
 		(dnp no)
-		(property "Reference" "C601"
+		(property "Reference" "C21"
 			(at 179.705 75.565 90)
 			(effects
@@
 		)
 		(instances
+			(project "GS"
+				(path "/4eb245a9-6c21-4f00-ae42-6a498711dd85/fd7daa6e-d3a6-4f28-bda8-c91b24a77464"
+					(reference "C21")
+					(unit 1)
+				)
+			)
 			(project "GS"
 				(path "/920f9ee9-d8de-4f24-ad72-1c45434a67fe/2c35cf26-1e44-42e5-8139-efbe5f54c1ed"
@@
 		(dnp no)
 		(fields_autoplaced yes)
-		(property "Reference" "#PWR0601"
+		(property "Reference" "#PWR064"
 			(at 190.5 74.93 0)
 			(effects
@@
 		)
 		(instances
+			(project "GS"
+				(path "/4eb245a9-6c21-4f00-ae42-6a498711dd85/fd7daa6e-d3a6-4f28-bda8-c91b24a77464"
+					(reference "#PWR064")
+					(unit 1)
+				)
+			)
 			(project "GS"
 				(path "/920f9ee9-d8de-4f24-ad72-1c45434a67fe/2c35cf26-1e44-42e5-8139-efbe5f54c1ed"
@@
 		(instances
 			(project "CMGFather"
+				(path "/4eb245a9-6c21-4f00-ae42-6a498711dd85/fd7daa6e-d3a6-4f28-bda8-c91b24a77464"
+					(reference "#PWR0104")
+					(unit 1)
+				)
+			)
+			(project "CMGFather"
 				(path "/9e354a01-2cea-4232-8b65-4471166b2c2b/7ef76fdd-30f3-4139-a072-8ee3fa540a64"
 					(reference "#PWR0104")
@@
 		(on_board yes)
 		(dnp no)
-		(property "Reference" "Y601"
+		(property "Reference" "Y1"
 			(at 173.355 89.535 90)
 			(effects
@@
 		(instances
 			(project "GS"
+				(path "/4eb245a9-6c21-4f00-ae42-6a498711dd85/fd7daa6e-d3a6-4f28-bda8-c91b24a77464"
+					(reference "Y1")
+					(unit 1)
+				)
+			)
+			(project "GS"
 				(path "/920f9ee9-d8de-4f24-ad72-1c45434a67fe/2c35cf26-1e44-42e5-8139-efbe5f54c1ed"

Commit message: 一旦回路図完成
Parts:
- renumbered BT101 to BT501, C21 to C501, C20 to C502, MICRO_SD1 to MICRO_SD501, U8 to U501, Y1 to Y501
Changed lines of the file:
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@@
 		(on_board yes)
 		(dnp no)
-		(property "Reference" "C20"
+		(property "Reference" "C502"
 			(at 140.97 85.725 0)
 			(effects
@@
 			(project "GS"
 				(path "/4eb245a9-6c21-4f00-ae42-6a498711dd85/fd7daa6e-d3a6-4f28-bda8-c91b24a77464"
-					(reference "C20")
+					(reference "C502")
 					(unit 1)
 				)
@@
 		(on_board yes)
 		(dnp no)
-		(property "Reference" "#PWR0606"
+		(property "Reference" "#PWR0505"
 			(at 228.6 90.17 0)
 			(effects
@@
 			(project "CMGFather"
 				(path "/4eb245a9-6c21-4f00-ae42-6a498711dd85/fd7daa6e-d3a6-4f28-bda8-c91b24a77464"
-					(reference "#PWR0606")
+					(reference "#PWR0505")
 					(unit 1)
 				)
@@
 		(dnp no)
 		(fields_autoplaced yes)
-		(property "Reference" "MICRO_SD1"
+		(property "Reference" "MICRO_SD501"
 			(at 117.475 76.2 0)
 			(effects
@@
 			(project "GS"
 				(path "/4eb245a9-6c21-4f00-ae42-6a498711dd85/fd7daa6e-d3a6-4f28-bda8-c91b24a77464"
-					(reference "MICRO_SD1")
+					(reference "MICRO_SD501")
 					(unit 1)
 				)
@@
 		(on_board yes)
 		(dnp no)
-		(property "Reference" "#PWR063"
+		(property "Reference" "#PWR0503"
 			(at 185.42 84.455 0)
 			(effects
@@
 			(project "GS"
 				(path "/4eb245a9-6c21-4f00-ae42-6a498711dd85/fd7daa6e-d3a6-4f28-bda8-c91b24a77464"
-					(reference "#PWR063")
+					(reference "#PWR0503")
 					(unit 1)
 				)
@@
 		(dnp no)
 		(fields_autoplaced yes)
-		(property "Reference" "#PWR065"
+		(property "Reference" "#PWR0507"
 			(at 190.5 107.315 0)
 			(effects
@@
 			(project "GS"
 				(path "/4eb245a9-6c21-4f00-ae42-6a498711dd85/fd7daa6e-d3a6-4f28-bda8-c91b24a77464"
-					(reference "#PWR065")
+					(reference "#PWR0507")
 					(unit 1)
 				)
@@
 		(dnp no)
 		(fields_autoplaced yes)
-		(property "Reference" "#PWR061"
+		(property "Reference" "#PWR0504"
 			(at 145.415 86.36 0)
 			(effects
@@
 			(project "GS"
 				(path "/4eb245a9-6c21-4f00-ae42-6a498711dd85/fd7daa6e-d3a6-4f28-bda8-c91b24a77464"
-					(reference "#PWR061")
+					(reference "#PWR0504")
 					(unit 1)
 				)
@@
 		(dnp no)
 		(fields_autoplaced yes)
-		(property "Reference" "BT101"
+		(property "Reference" "BT501"
 			(at 232.41 78.1684 0)
 			(effects
@@
 			(project "CMGFather"
 				(path "/4eb245a9-6c21-4f00-ae42-6a498711dd85/fd7daa6e-d3a6-4f28-bda8-c91b24a77464"
-					(reference "BT101")
+					(reference "BT501")
 					(unit 1)
 				)
@@
 		(dnp no)
 		(fields_autoplaced yes)
-		(property "Reference" "U8"
+		(property "Reference" "U501"
 			(at 192.6941 78.105 0)
 			(effects
@@
 			(project "GS"
 				(path "/4eb245a9-6c21-4f00-ae42-6a498711dd85/fd7daa6e-d3a6-4f28-bda8-c91b24a77464"
-					(reference "U8")
+					(reference "U501")
 					(unit 1)
 				)
@@
 		(dnp no)
 		(fields_autoplaced yes)
-		(property "Reference" "#PWR062"
+		(property "Reference" "#PWR0506"
 			(at 145.415 106.68 0)
 			(effects
@@
 			(project "GS"
 				(path "/4eb245a9-6c21-4f00-ae42-6a498711dd85/fd7daa6e-d3a6-4f28-bda8-c91b24a77464"
-					(reference "#PWR062")
+					(reference "#PWR0506")
 					(unit 1)
 				)
@@
 		(on_board yes)
 		(dnp no)
-		(property "Reference" "C21"
+		(property "Reference" "C501"
 			(at 179.705 75.565 90)
 			(effects
@@
 			(project "GS"
 				(path "/4eb245a9-6c21-4f00-ae42-6a498711dd85/fd7daa6e-d3a6-4f28-bda8-c91b24a77464"
-					(reference "C21")
+					(reference "C501")
 					(unit 1)
 				)
@@
 		(dnp no)
 		(fields_autoplaced yes)
-		(property "Reference" "#PWR064"
+		(property "Reference" "#PWR0501"
 			(at 190.5 74.93 0)
 			(effects
@@
 			(project "GS"
 				(path "/4eb245a9-6c21-4f00-ae42-6a498711dd85/fd7daa6e-d3a6-4f28-bda8-c91b24a77464"
-					(reference "#PWR064")
+					(reference "#PWR0501")
 					(unit 1)
 				)
@@
 		(dnp no)
 		(fields_autoplaced yes)
-		(property "Reference" "#PWR0104"
+		(property "Reference" "#PWR0502"
 			(at 228.6 77.47 0)
 			(effects
@@
 			(project "CMGFather"
 				(path "/4eb245a9-6c21-4f00-ae42-6a498711dd85/fd7daa6e-d3a6-4f28-bda8-c91b24a77464"
-					(reference "#PWR0104")
+					(reference "#PWR0502")
 					(unit 1)
 				)
@@
 		(on_board yes)
 		(dnp no)
-		(property "Reference" "Y1"
+		(property "Reference" "Y501"
 			(at 173.355 89.535 90)
 			(effects
@@
 			(project "GS"
 				(path "/4eb245a9-6c21-4f00-ae42-6a498711dd85/fd7daa6e-d3a6-4f28-bda8-c91b24a77464"
-					(reference "Y1")
-					(unit 1)
-				)
+					(reference "Y501")
+					(unit 1)
+				)

Commit message: LogicBoard一旦完成
Parts:
- removed BT501: Battery_Cell, WOBCLibrary:cr1220, symbol Device:Battery_Cell
- removed C501: 100nF, Capacitor_SMD:C_0402_1005Metric, symbol Device:C_Small
- removed U501: PCF8563T, Package_SO:SOIC-8_3.9x4.9mm_P1.27mm, symbol Timer_RTC:PCF8563T
- removed Y501: Crystal, Crystal:Crystal_SMD_3215-2Pin_3.2x1.5mm, symbol Device:Crystal
Connections:
- no-connect marks 4 -> 2
Other:
- note removed: "I2C ADDR: 0x51"
- note removed: "RTC"

Commit message: 途中
Parts:
- C501: renamed from C502; footprint Capacitor_SMD:C_0402_1005Metric -> Capacitor_SMD:C_0603_1608Metric
Changed lines of the file:
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@@
 		(on_board yes)
 		(dnp no)
-		(property "Reference" "C502"
+		(property "Reference" "C501"
 			(at 140.97 85.725 0)
 			(effects
@@
 			)
 		)
-		(property "Footprint" "Capacitor_SMD:C_0402_1005Metric"
+		(property "Footprint" "Capacitor_SMD:C_0603_1608Metric"
 			(at 145.415 86.995 0)
 			(effects
@@
 			(project "GS"
 				(path "/4eb245a9-6c21-4f00-ae42-6a498711dd85/fd7daa6e-d3a6-4f28-bda8-c91b24a77464"
-					(reference "C502")
+					(reference "C501")
 					(unit 1)
 				)
@@
 		(dnp no)
 		(fields_autoplaced yes)
-		(property "Reference" "#PWR0504"
+		(property "Reference" "#PWR0501"
 			(at 145.415 86.36 0)
 			(effects
@@
 			(project "GS"
 				(path "/4eb245a9-6c21-4f00-ae42-6a498711dd85/fd7daa6e-d3a6-4f28-bda8-c91b24a77464"
-					(reference "#PWR0504")
+					(reference "#PWR0501")
 					(unit 1)
 				)
@@
 		(dnp no)
 		(fields_autoplaced yes)
-		(property "Reference" "#PWR0506"
+		(property "Reference" "#PWR0502"
 			(at 145.415 106.68 0)
 			(effects
@@
 			(project "GS"
 				(path "/4eb245a9-6c21-4f00-ae42-6a498711dd85/fd7daa6e-d3a6-4f28-bda8-c91b24a77464"
-					(reference "#PWR0506")
-					(unit 1)
-				)
+					(reference "#PWR0502")
+					(unit 1)
+				)
