File: hardware/modules/CMG/CMGSon/MotorControl.kicad_sch (KiCad schematic)
At the start: 18 parts, among them J1 MotorDriver, J2 ch1, J3 ch2, U1 LM2903PWR

Commit message: コンポーネントを配置 サーボコンポーネントを追加
Parts:
- added C402: 10uF, Capacitor_SMD:C_0603_1608Metric, symbol Device:C_Small
- added C403: 100n, Capacitor_SMD:C_0402_1005Metric, symbol Device:C_Small
- added J403: LiPo_{in}, Connector_AMASS:AMASS_XT30PW-M_1x02_P2.50mm_Horizontal, symbol Connector_Generic:Conn_01x02
- added J404: LiPo_{out}, Connector_AMASS:AMASS_XT30PW-M_1x02_P2.50mm_Horizontal, symbol Connector_Generic:Conn_01x02
- added R402: 3mΩ, Resistor_SMD:R_2010_5025Metric, symbol Device:R
- added U401: INA226, Package_SO:VSSOP-10_3x3mm_P0.5mm, symbol Sensor_Energy:INA226
Connections:
- net GND: now also C402.2, C403.2, J403.2 (Pin_2), J404.2 (Pin_2), U401.7 (GND)
- net VDD: now also C402.1, C403.1, U401.1 (A1), U401.6 (VS)
- new net: J403.1 (Pin_1), R402.2, U401.10 (Vin+), U401.8 (Vbus)
- new net I2C_SCL: U401.2 (A0), U401.5 (SCL)
- new net I2C_SDA: U401.4 (SDA)
- new net LiPo_{out}: J404.1 (Pin_1), R402.1, U401.9 (Vin-)
- no-connect marks 0 -> 1
Other:
- note added: "I2C ADDR : 0x47"
- note added: "PowerMeasure"
- note added: "Tachometer"
- note removed: "Tacchometer"
- moved on the sheet: C105, C106, C901, C902, C903, C904, J1, J2, J3, R1, R115, R2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

Commit message: 一旦回路図完成
Parts:
- renumbered C105 to C401, C106 to C402, C402 to C403, C403 to C404, C901 to C405, C902 to C406, C903 to C407, C904 to C408, J403 to J401, J2 to J402, J3 to J403, J1 to J405, R2 to R401, R3 to R402, R901 to R403, R902 to R404, R1 to R405, R402 to R406, R115 to R407, RV101 to RV401, RV102 to RV402, U1 to U401, U401 to U402

Commit message: 途中
Parts:
- J402, J403: footprint Connector_JST:JST_PH_S3B-PH-K_1x03_P2.00mm_Horizontal -> Connector_JST:JST_PH_B3B-PH-K_1x03_P2.00mm_Vertical
- J405: footprint Connector_JST:JST_XA_S05B-XASK-1_1x05_P2.50mm_Horizontal -> Connector_JST:JST_PH_B5B-PH-K_1x05_P2.00mm_Vertical
Connections:
- net GND: now also J401.1 (Pin_2), J404.1 (Pin_2); no longer J401.2 (Pin_2), J404.2 (Pin_2)
- net LiPo_{out}: now also J404.2 (Pin_1); no longer J404.1 (Pin_1)
- net at R406.2, U402.10 (Vin+), U402.8 (Vbus): now also J401.2 (Pin_1); no longer J401.1 (Pin_1)
Changed lines of the file:
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@@
 			)
 		)
-		(property "Footprint" "Connector_JST:JST_PH_S3B-PH-K_1x03_P2.00mm_Horizontal"
+		(property "Footprint" "Connector_JST:JST_PH_B3B-PH-K_1x03_P2.00mm_Vertical"
 			(at 83.82 121.92 0)
 			(effects
@@
 			)
 		)
-		(property "Footprint" "Connector_JST:JST_XA_S05B-XASK-1_1x05_P2.50mm_Horizontal"
+		(property "Footprint" "Connector_JST:JST_PH_B5B-PH-K_1x05_P2.00mm_Vertical"
 			(at 68.58 168.91 0)
 			(effects
@@
 	)
 	(symbol
+		(lib_name "Conn_01x02_1")
 		(lib_id "Connector_Generic:Conn_01x02")
 		(at 252.73 125.73 0)
@@
 			)
 		)
-		(property "Footprint" "Connector_JST:JST_PH_S3B-PH-K_1x03_P2.00mm_Horizontal"
+		(property "Footprint" "Connector_JST:JST_PH_B3B-PH-K_1x03_P2.00mm_Vertical"
 			(at 121.92 121.92 0)
 			(effects
