File: hardware/modules/CMG/CMGFather/Logger.kicad_sch (KiCad schematic)
At the start: 6 parts, among them U601 PCF8563T, Y601 Crystal

Commit message: LogicBoard一旦完成
Parts:
- removed BT101: Battery_Cell, WOBCLibrary:cr1220, symbol Device:Battery_Cell
Connections:
- net +BATT is gone; now on net VDD: C601.2, U601.8 (VDD)

Commit message: 一旦完成
Parts:
- C602: footprint Capacitor_SMD:C_0402_1005Metric -> Capacitor_SMD:C_0603_1608Metric
Changed lines of the file:
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@@
 			)
 		)
-		(property "Footprint" "Capacitor_SMD:C_0402_1005Metric"
+		(property "Footprint" "Capacitor_SMD:C_0603_1608Metric"
 			(at 145.415 86.995 0)
 			(effects
