File: hardware/modules/Separation/LiPoPower.kicad_sch (KiCad schematic)
At the start: 53 parts, among them J1 Battery, J2 Ext Switch, J4 LiPo, SW2 Power Switch, U10 INA226, U302 TPS2116DRL, U6 MCP73871-1CC, U7 INA226, U9 TPS63070RNMR

Commit message: 一旦
Parts:
- renumbered C7 to C801, C8 to C802, C12 to C803, C13 to C804, C14 to C805, C302 to C806, C314 to C807, C308 to C808, C11 to C809, C9 to C810, C10 to C811, C312 to C812, C7 to C813, C7 to C814, C7 to C815, C307 to C816, F301 to F801, F1 to F802, F3 to F803, J1 to J801, J2 to J802, J4 to J803, L1 to L801, LED301 to LED801, LED5 to LED802, LED1 to LED803, LED3 to LED804, R21 to R801, R21 to R802, R20 to R803, R13 to R804, R19 to R805, R306 to R806, R18 to R807, R22 to R808, R309 to R809, R15 to R810, R311 to R811, R8 to R812, R16 to R813, R8 to R814, R9 to R815, R10 to R816, R317 to R817, R14 to R818, RV1 to RV801, SW2 to SW801, U9 to U801, U302 to U802, U10 to U803, U10 to U804, U6 to U805, U7 to U806
