File: hardware/modules/Separation/Logger.kicad_sch (KiCad schematic)
At the start: 5 parts, among them U8 PCF8563T, Y1 Crystal

Commit message: 一旦
Parts:
- C602: renamed from C20; footprint Capacitor_SMD:C_0402_1005Metric -> Capacitor_SMD:C_0603_1608Metric
- renumbered C21 to C601, MICRO_SD1 to MICRO_SD601, U8 to U601, Y1 to Y601
Changed lines of the file:
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@@
 		(on_board yes)
 		(dnp no)
-		(property "Reference" "C20"
+		(property "Reference" "C602"
 			(at 140.97 85.725 0)
 			(effects
@@
 			)
 		)
-		(property "Footprint" "Capacitor_SMD:C_0402_1005Metric"
+		(property "Footprint" "Capacitor_SMD:C_0603_1608Metric"
 			(at 145.415 86.995 0)
 			(effects
@@
 			(project "GS"
 				(path "/67e7b825-e210-4fbd-ae56-bcf369c4487b/fdbc0a00-550f-4f67-9e49-89def436726b"
-					(reference "C20")
+					(reference "C602")
 					(unit 1)
 				)
@@
 		(dnp no)
 		(fields_autoplaced yes)
-		(property "Reference" "MICRO_SD1"
+		(property "Reference" "MICRO_SD601"
 			(at 117.475 76.2 0)
 			(effects
@@
 			(project "GS"
 				(path "/67e7b825-e210-4fbd-ae56-bcf369c4487b/fdbc0a00-550f-4f67-9e49-89def436726b"
-					(reference "MICRO_SD1")
+					(reference "MICRO_SD601")
 					(unit 1)
 				)
@@
 		(on_board yes)
 		(dnp no)
-		(property "Reference" "#PWR063"
+		(property "Reference" "#PWR0602"
 			(at 185.42 84.455 0)
 			(effects
@@
 			(project "GS"
 				(path "/67e7b825-e210-4fbd-ae56-bcf369c4487b/fdbc0a00-550f-4f67-9e49-89def436726b"
-					(reference "#PWR063")
+					(reference "#PWR0602")
 					(unit 1)
 				)
@@
 		(dnp no)
 		(fields_autoplaced yes)
-		(property "Reference" "#PWR0301"
+		(property "Reference" "#PWR0601"
 			(at 190.5 74.93 0)
 			(effects
@@
 			(project ""
 				(path "/67e7b825-e210-4fbd-ae56-bcf369c4487b/fdbc0a00-550f-4f67-9e49-89def436726b"
-					(reference "#PWR0301")
+					(reference "#PWR0601")
 					(unit 1)
 				)
@@
 		(dnp no)
 		(fields_autoplaced yes)
-		(property "Reference" "#PWR065"
+		(property "Reference" "#PWR0605"
 			(at 190.5 107.315 0)
 			(effects
@@
 			(project "GS"
 				(path "/67e7b825-e210-4fbd-ae56-bcf369c4487b/fdbc0a00-550f-4f67-9e49-89def436726b"
-					(reference "#PWR065")
+					(reference "#PWR0605")
 					(unit 1)
 				)
@@
 		(dnp no)
 		(fields_autoplaced yes)
-		(property "Reference" "#PWR061"
+		(property "Reference" "#PWR0603"
 			(at 145.415 86.36 0)
 			(effects
@@
 			(project "GS"
 				(path "/67e7b825-e210-4fbd-ae56-bcf369c4487b/fdbc0a00-550f-4f67-9e49-89def436726b"
-					(reference "#PWR061")
+					(reference "#PWR0603")
 					(unit 1)
 				)
@@
 		(dnp no)
 		(fields_autoplaced yes)
-		(property "Reference" "U8"
+		(property "Reference" "U601"
 			(at 192.6941 78.105 0)
 			(effects
@@
 			(project "GS"
 				(path "/67e7b825-e210-4fbd-ae56-bcf369c4487b/fdbc0a00-550f-4f67-9e49-89def436726b"
-					(reference "U8")
+					(reference "U601")
 					(unit 1)
 				)
@@
 		(dnp no)
 		(fields_autoplaced yes)
-		(property "Reference" "#PWR062"
+		(property "Reference" "#PWR0604"
 			(at 145.415 106.68 0)
 			(effects
@@
 			(project "GS"
 				(path "/67e7b825-e210-4fbd-ae56-bcf369c4487b/fdbc0a00-550f-4f67-9e49-89def436726b"
-					(reference "#PWR062")
+					(reference "#PWR0604")
 					(unit 1)
 				)
@@
 		(on_board yes)
 		(dnp no)
-		(property "Reference" "C21"
+		(property "Reference" "C601"
 			(at 179.705 75.565 90)
 			(effects
@@
 			(project "GS"
 				(path "/67e7b825-e210-4fbd-ae56-bcf369c4487b/fdbc0a00-550f-4f67-9e49-89def436726b"
-					(reference "C21")
+					(reference "C601")
 					(unit 1)
 				)
@@
 		(on_board yes)
 		(dnp no)
-		(property "Reference" "Y1"
+		(property "Reference" "Y601"
 			(at 173.355 89.535 90)
 			(effects
@@
 			(project "GS"
 				(path "/67e7b825-e210-4fbd-ae56-bcf369c4487b/fdbc0a00-550f-4f67-9e49-89def436726b"
-					(reference "Y1")
-					(unit 1)
-				)
+					(reference "Y601")
+					(unit 1)
+				)
