File: hardware/modules/Separation/Nichrome.kicad_sch (KiCad schematic)
At the start: 34 parts, among them J201 LiPo 3 Cell, J202 IGNITER, J203 PowerSW, J804 LaunchDetection, Q201 Q_PMOS_GSD, Q202 Q_NMOS_DGS, Q203 Q_NPN_BEC, Q804 NMOS, U201 INA226

Commit message: 回路図一旦
Other:
- note removed: "←そもそもこれは何用のダイオードなんですか？"
Changed lines of the file:
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@@
-		)
-	)
-	(text "←そもそもこれは何用のダイオードなんですか？"
-		(exclude_from_sim no)
-		(at 163.83 139.954 0)
-		(effects
-			(font
-				(size 1.27 1.27)
-			)
-			(justify left)
 		)
 	)

Commit message: 一旦
Parts:
- renumbered BZ201 to BZ501, C201 to C501, C202 to C502, D201 to D501, D206 to D502, D203 to D503, D202 to D504, D204 to D505, D205 to D506, D807 to D507, F201 to F501, J201 to J501, J203 to J502, J202 to J503, J804 to J504, Q201 to Q501, Q203 to Q502, Q202 to Q503, Q804 to Q504, R204 to R501, R206 to R502, R210 to R503, R201 to R504, R211 to R505, R202 to R506, R203 to R507, R207 to R508, R209 to R509, R810 to R510, R208 to R511, R205 to R512, R813 to R513, R814 to R514, U201 to U501
