File: hardware/modules/Separation/GPSActive.kicad_sch (KiCad schematic)
At the start: 15 parts, among them J701 SMA, U701 NEO-M9N-00B

Commit message: 修正
Parts:
- USB701: LCSC C2982481 -> C720625
Other:
- moved on the sheet: R704, R705
Changed lines of the file:
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@@
-	(wire
-		(pts
-			(xy 215.9 92.71) (xy 215.9 91.44)
-		)
-		(stroke
-			(width 0)
-			(type default)
-		)
-	)
 	(wire
 		(pts
@@
 	(wire
 		(pts
-			(xy 223.52 93.98) (xy 228.6 93.98)
+			(xy 224.79 92.71) (xy 228.6 92.71)
+		)
+		(stroke
+			(width 0)
+			(type default)
+		)
+	)
+	(wire
+		(pts
+			(xy 224.79 95.25) (xy 228.6 95.25)
 		)
 		(stroke
@@
 	(wire
 		(pts
-			(xy 212.09 92.71) (xy 215.9 92.71)
+			(xy 212.09 92.71) (xy 217.17 92.71)
 		)
 		(stroke
@@
 	(wire
 		(pts
-			(xy 217.17 93.98) (xy 215.9 93.98)
-		)
-		(stroke
-			(width 0)
-			(type default)
-		)
-	)
-	(wire
-		(pts
 			(xy 135.89 113.03) (xy 111.76 113.03)
 		)
@@
 	(wire
 		(pts
-			(xy 223.52 91.44) (xy 228.6 91.44)
-		)
-		(stroke
-			(width 0)
-			(type default)
-		)
-	)
-	(wire
-		(pts
 			(xy 76.2 96.52) (xy 76.2 97.79)
-		)
-		(stroke
-			(width 0)
-			(type default)
-		)
-	)
-	(wire
-		(pts
-			(xy 217.17 95.25) (xy 217.17 93.98)
 		)
 		(stroke
@@
 	(hierarchical_label "TX"
 		(shape output)
-		(at 228.6 93.98 0)
+		(at 228.6 95.25 0)
 		(effects
 			(font
@@
 	(hierarchical_label "RX"
 		(shape input)
-		(at 228.6 91.44 0)
+		(at 228.6 92.71 0)
 		(effects
 			(font
@@
 			)
 		)
-		(property "LCSC" "C2982481"
+		(property "LCSC" "C720625"
 			(at 50.8 93.98 0)
 			(effects
@@
 	(symbol
 		(lib_id "Device:R")
-		(at 219.71 93.98 270)
+		(at 220.98 95.25 270)
 		(unit 1)
 		(exclude_from_sim no)
@@
 		(dnp no)
 		(property "Reference" "R705"
-			(at 225.552 94.996 90)
+			(at 226.822 96.266 90)
 			(effects
 				(font
@@
 		)
 		(property "Value" "33"
-			(at 215.138 94.742 90)
+			(at 216.408 96.012 90)
 			(effects
 				(font
@@
 		)
 		(property "Footprint" "Resistor_SMD:R_0402_1005Metric"
-			(at 219.71 92.202 90)
+			(at 220.98 93.472 90)
 			(effects
 				(font
@@
 		)
 		(property "Datasheet" "~"
-			(at 219.71 93.98 0)
+			(at 220.98 95.25 0)
 			(effects
 				(font
@@
 		)
 		(property "Description" ""
-			(at 219.71 93.98 0)
+			(at 220.98 95.25 0)
 			(effects
 				(font
@@
 		)
 		(property "LCSC" "C25105"
-			(at 219.71 93.98 0)
+			(at 220.98 95.25 0)
 			(effects
 				(font
@@
 		)
 		(property "Sim.Device" ""
-			(at 219.71 93.98 0)
+			(at 220.98 95.25 0)
 			(effects
 				(font
@@
 		)
 		(property "Sim.Pins" ""
-			(at 219.71 93.98 0)
+			(at 220.98 95.25 0)
 			(effects
 				(font
@@
 	(symbol
 		(lib_id "Device:R")
-		(at 219.71 91.44 270)
+		(at 220.98 92.71 270)
 		(unit 1)
 		(exclude_from_sim no)
@@
 		(dnp no)
 		(property "Reference" "R704"
-			(at 225.552 91.948 90)
+			(at 226.822 93.218 90)
 			(effects
 				(font
@@
 		)
 		(property "Value" "33"
-			(at 215.138 92.456 90)
+			(at 216.408 93.726 90)
 			(effects
 				(font
@@
 		)
 		(property "Footprint" "Resistor_SMD:R_0402_1005Metric"
-			(at 219.71 89.662 90)
+			(at 220.98 90.932 90)
 			(effects
 				(font
@@
 		)
 		(property "Datasheet" "~"
-			(at 219.71 91.44 0)
+			(at 220.98 92.71 0)
 			(effects
 				(font
@@
 		)
 		(property "Description" ""
-			(at 219.71 91.44 0)
+			(at 220.98 92.71 0)
 			(effects
 				(font
@@
 		)
 		(property "LCSC" "C25105"
-			(at 219.71 91.44 0)
+			(at 220.98 92.71 0)
 			(effects
 				(font
@@
 		)
 		(property "Sim.Device" ""
-			(at 219.71 91.44 0)
+			(at 220.98 92.71 0)
 			(effects
 				(font
@@
 		)
 		(property "Sim.Pins" ""
-			(at 219.71 91.44 0)
-			(effects
-				(font
+			(at 220.98 92.71 0)
+			(effects
+				(font
