File: hardware/modules/GS2026/GS2026.kicad_pcb (KiCad board)
At the start: 2 copper layers, 120 x 60 mm, 38 parts, among them J301 Jumper, J302 Conn_01x04_MountingPin, J401 Jumper, J402 Conn_01x04_MountingPin, SW201 RESET_sw, SW501 sw1, U101 AMS1117-3.3, U201 TPS3820, U202 SN65HVD230, U203 ESP32-S3-WROOM-1

Commit message: 途中
Parts:
- C101, C201, C202, C301, C401, D206, R203, R204, R205, R206, R301, R401, SW201, U101, U201, U202: moved to B.Cu
- moved SW501 135.5 mm to (173.1, 72.4)
- moved C101 87.9 mm to (160.0, 76.2), turned to 90 degrees
- moved C102 86.8 mm to (155.7, 68.6)
- turned C201 to 180 degrees
- turned C301 to 180 degrees
- turned C401 to 180 degrees
- turned R301 to 180 degrees
- turned R401 to 180 degrees
- turned SW201 to 180 degrees
- turned U101 to 180 degrees
- turned U201 to 180 degrees
- turned U202 to 180 degrees

Commit message: ブートボタンの設置と配置完了
Parts:
- added C601: 10uF, Capacitor_SMD:C_0402_1005Metric, B.Cu at (143.5, 76.6)
- added C602: 100nF, Capacitor_SMD:C_0402_1005Metric, B.Cu at (163.7, 76.2)
- added MICRO_SD601: TF-01A, WOBCLibrary:TF-01A, B.Cu at (141.5, 86.1)
- added SW202: RESET, WOBCLibrary:TVAF06-A020B-R, B.Cu at (130.2, 59.3)
- added U601: PCF8563T, Package_SO:SOIC-8_3.9x4.9mm_P1.27mm, B.Cu at (159.3, 80.0)
- added Y601: Crystal, Crystal:Crystal_SMD_3215-2Pin_3.2x1.5mm, B.Cu at (153.6, 81.3)
- C203, C204, D201, D202, D203, D204, D205, R201, R202, R207, USB201: moved to B.Cu
- moved R502 136.8 mm to (174.8, 64.6), turned to 90 degrees
- moved C203 128.3 mm to (154.6, 45.7), turned to -90 degrees
- moved C204 126.5 mm to (153.0, 45.7), turned to -90 degrees
- moved D205 121.0 mm to (129.8, 54.5), turned to 90 degrees
- moved D204 97.5 mm to (174.1, 56.8), turned to -90 degrees
- moved D203 80.1 mm to (169.6, 86.5)
- moved D202 79.1 mm to (167.8, 86.5)
- moved R501 78.9 mm to (72.9, 73.7), turned to 90 degrees
- moved D201 75.2 mm to (171.5, 86.5), turned to 180 degrees
- moved R207 70.3 mm to (154.2, 57.1), turned to 90 degrees
- moved SW501 25.7 mm to (157.6, 92.9), turned to -90 degrees
- moved C101 6.53 mm to (154.9, 72.1)
- moved U101 6.32 mm to (148.9, 70.8)
- moved R203 1.12 mm to (172.5, 56.7)
- moved R202 0.68 mm to (166.4, 84.8), turned to 180 degrees
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Connections:
- C102 pad 1: VDD -> GND
- C201 pad 2: VDD -> GND
- C202 pad 2: VDD -> GND
- C203 pad 2: VDD -> GND
- C204 pad 1: VDD -> GND
- C301 pad 2: VDD -> GND
- C401 pad 2: VDD -> GND
- J302 pad 3: VDD -> GND
- J402 pad 3: VDD -> GND
- R203 pad 1: VDD -> GND
- R205 pad 1: VDD -> GND
- R207 pad 1: VDD -> GND
- U101 pad 2: VDD -> GND
- U201 pad 5: VDD -> GND
- U202 pad 3: VDD -> GND
- U203 pad 2: VDD -> GND
- U203 pad 27: unconnected-(U203-GPIO0/BOOT-Pad27) -> Net-(U203-GPIO0/BOOT)
- lcd501 pad 2: VDD -> GND

Commit message: 一旦あきらめる
Parts:
- C102, R501, R502: moved to B.Cu
- moved C102 1.10 mm to (154.6, 68.7), turned to 90 degrees
- moved R502 0.85 mm to (175.6, 64.2)
- moved C101 0.49 mm to (154.4, 72.0)
Routing:
- net Net-(lcd501-Vo): track 0.00 -> 3.59 mm

Commit message: 一旦
Routing:
- net GND: track 0.00 -> 3.33 mm
Changed lines of the file:
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@@
+	)
+	(segment
+		(start 69.79 74.695)
+		(end 72.456 74.695)
+		(width 1)
+		(layer "B.Cu")
+		(net 1)
+	)
+	(segment
+		(start 72.456 74.695)
+		(end 72.925 74.226)
+		(width 1)
+		(layer "B.Cu")
+		(net 1)
 	)
 	(segment

Commit message: 途中経過
Parts:
- moved C101 17.1 mm to (171.3, 69.1)
- moved C102 17.1 mm to (171.4, 65.8)
- moved U101 17.1 mm to (165.8, 67.9)
- moved U601 12.7 mm to (151.8, 69.8)
- moved Y601 12.7 mm to (146.0, 71.1)
- moved C202 10.1 mm to (126.0, 50.4)
- moved C602 7.42 mm to (157.4, 72.3), turned to -90 degrees
- moved D203 0.54 mm to (169.4, 86.0), turned to -90 degrees
- moved R202 0.40 mm to (166.1, 84.8)
- moved D201 0.23 mm to (171.5, 86.2)
- moved D202 0.18 mm to (167.7, 86.5), turned to -90 degrees
Routing:
- net GND: track 3.33 -> 171.9 mm, vias 0 -> 2
- net Net-(SW501-B): track 0.00 -> 41.8 mm
- net (no net): track 0.00 -> 35.6 mm
- net RESET: track 0.00 -> 29.6 mm
- net /ESP32S3/WDI: track 0.00 -> 27.6 mm, vias 0 -> 2
- net /ESP32S3/I2C_SCL: track 0.00 -> 23.1 mm
- net /ESP32S3/I2C_SDA: track 0.00 -> 17.9 mm
- net /CAN/CANL: track 0.00 -> 14.0 mm
- net VBUS: track 0.00 -> 11.0 mm
- net Net-(U201-MR): track 0.00 -> 7.46 mm
- net /CAN/CANH: track 0.00 -> 7.30 mm
- net /ESP32S3/USB_D-: track 0.00 -> 6.82 mm
- net Net-(lcd501-A): track 0.00 -> 4.78 mm
- net Net-(USB201-CC1): track 0.00 -> 4.33 mm
- net Net-(J401-Pin_1): track 0.00 -> 3.95 mm
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
Commit message: 配線完了
Parts:
- moved C601 1.79 mm to (143.6, 74.8), turned to 0 degrees
- turned C201 to 0 degrees
- turned C204 to 90 degrees
Connections:
- C102 pad 1: GND -> VDD
- C201 pad 2: GND -> VDD
- C202 pad 2: GND -> VDD
- C203 pad 2: GND -> VDD
- C204 pad 1: GND -> VDD
- C301 pad 2: GND -> VDD
- C401 pad 2: GND -> VDD
- C601 pad 1: GND -> VDD
- J302 pad 3: GND -> VDD
- J402 pad 3: GND -> VDD
- MICRO_SD601 pad 4: GND -> VDD
- R203 pad 1: GND -> VDD
- R205 pad 1: GND -> VDD
- R207 pad 1: GND -> VDD
- U101 pad 2: GND -> VDD
- U201 pad 5: GND -> VDD
- U202 pad 3: GND -> VDD
- U203 pad 2: GND -> VDD
- lcd501 pad 2: GND -> VDD
Routing:
- net GND: track 171.9 -> 311.5 mm, vias 2 -> 5
- net /CAN/CANH: track 7.30 -> 92.6 mm
- net VDD: track 0.00 -> 85.1 mm, vias 0 -> 7
- net /CAN/CANL: track 14.0 -> 66.8 mm
- net /ESP32S3/GPIO13: track 0.00 -> 19.4 mm, vias 0 -> 2
- net /ESP32S3/GPIO10/ADC1_CH9: track 0.00 -> 18.0 mm
- net /ESP32S3/GPIO12: track 0.00 -> 17.4 mm
- net /ESP32S3/GPIO11: track 0.00 -> 17.1 mm, vias 0 -> 2
- net /ESP32S3/GPIO9/ADC1_CH8: track 0.00 -> 16.7 mm, vias 0 -> 2
- net /ESP32S3/CAN_RX: track 0.00 -> 14.9 mm
- net /ESP32S3/CAN_TX: track 0.00 -> 12.7 mm
- net /ESP32S3/VUSB: track 2.12 -> 11.7 mm
- net VBUS: track 11.0 -> 11.7 mm

Commit message: 修正
Routing:
- net GND: track 311.5 -> 359.9 mm, vias 5 -> 8
- net /CAN/CANH: track 92.6 -> 117.2 mm, vias 0 -> 2
- net /CAN/CANL: track 66.8 -> 91.1 mm, vias 0 -> 2
- net VDD: track 85.1 -> 94.8 mm, vias 7 -> 8

Commit message: あと少し
Parts:
- moved J301 3.00 mm to (92.9, 78.3), turned to -90 degrees
- moved J401 2.97 mm to (107.2, 77.2), turned to -90 degrees
- moved R401 2.16 mm to (105.2, 80.0)
- moved R301 1.61 mm to (90.5, 80.5)
Connections:
- D201 pad 2: /ESP32S3/VUSB -> VBUS
- USB201 pad A4: /ESP32S3/VUSB -> VBUS
- USB201 pad A9: /ESP32S3/VUSB -> VBUS
- USB201 pad B4: /ESP32S3/VUSB -> VBUS
- USB201 pad B9: /ESP32S3/VUSB -> VBUS
- lcd501 pad 13: /ESP32S3/GPIO18 -> /ESP32S3/GPIO5/ADC1_CH4
- lcd501 pad 14: /ESP32S3/GPIO8/ADC1_CH7 -> /ESP32S3/GPIO4/ADC1_CH3
- lcd501 pad 4: /ESP32S3/GPIO4/ADC1_CH3 -> /ESP32S3/GPIO8/ADC1_CH7
- lcd501 pad 6: /ESP32S3/GPIO5/ADC1_CH4 -> /ESP32S3/GPIO18
- lcd501 pad GND: (no net) -> GND
Routing:
- net VDD: track 94.8 -> 225.8 mm, vias 8 -> 11
- net /ESP32S3/USB_D-: track 6.82 -> 41.3 mm, vias 0 -> 2
- net /ESP32S3/USB_D+: track 3.78 -> 36.8 mm, vias 0 -> 2
- net VBUS: track 11.7 -> 40.5 mm, vias 0 -> 2
- net /CAN/CANH: track 117.2 -> 92.4 mm, vias 2 -> 0
- net /ESP32S3/VUSB: track 11.7 -> 0.00 mm
- net GND: track 359.9 -> 362.0 mm, vias 8 -> 9
- net /CAN/CANL: track 91.1 -> 90.3 mm
- net Net-(J401-Pin_1): track 3.95 -> 3.38 mm, vias 0 -> 1
- net Net-(J301-Pin_1): track 3.51 -> 3.02 mm, vias 0 -> 1
