File: hardware/modules/LoRa2026/LoRa2.kicad_sch (KiCad schematic)
At the start: 13 parts, among them J203 SMA, J204 SMA, U202 E220-900T22S(JP)

Commit message: LoRa2026修正ver2
Parts:
- removed C204, C205, C208: 100p, Capacitor_SMD:C_0603_1608Metric, symbol Device:C_Small
- removed C206, C207, C210: 100n, Capacitor_SMD:C_0402_1005Metric, symbol Device:C_Small
- removed C209: 10u, Capacitor_SMD:C_0603_1608Metric, symbol Device:C_Small
- removed D201, D202: ESD9B5.0ST5G, Diode_SMD:D_SOD-882, symbol Diode:ESD9B5.0ST5G
- removed J203, J204: SMA, WOBCLibrary:SMA_aki, symbol Connector:Conn_Coaxial_Power
- removed Switch201: XA17-G4K1, Package_TO_SOT_SMD:SOT-363_SC-70-6, symbol XA17-G4K:XA17-G4K
- removed U202: E220-900T22S(JP), WOBCLibrary:E220-900T22S(JP), symbol RF_Module_additional:E220-900T22S(JP)
- added C401, C402, C405: 100p, Capacitor_SMD:C_0603_1608Metric, symbol Device:C_Small
- added C403, C404, C407: 100n, Capacitor_SMD:C_0402_1005Metric, symbol Device:C_Small
- added C406: 10u, Capacitor_SMD:C_0603_1608Metric, symbol Device:C_Small
- added D401, D402: ESD9B5.0ST5G, Diode_SMD:D_SOD-882, symbol Diode:ESD9B5.0ST5G
- added J401, J402: SMA, WOBCLibrary:SMA_aki, symbol Connector:Conn_Coaxial_Power
- added Switch401: XA17-G4K1, Package_TO_SOT_SMD:SOT-363_SC-70-6, symbol XA17-G4K:XA17-G4K
- added U401: E220-900T22S(JP), WOBCLibrary:E220-900T22S(JP), symbol RF_Module_additional:E220-900T22S(JP)
Connections:
- net GND: now also C403.2, C404.2, C406.2, C407.2, D401.1 (A1), D402.1 (A1), J401.2 (Ext), J402.2 (Ext), Switch401.2 (GND), U401.1 (GND), U401.11 (GND), U401.13 (GND), U401.19 (GND), U401.2 (GND), U401.20 (GND), U401.22 (GND), U401.3 (GND), U401.4 (GND)
- net LoRa_AUX: now also U401.9 (AUX)
- net LoRa_M0: now also U401.5 (M0)
- net LoRa_M1: now also U401.6 (M1)
- net LoRa_RTX: now also U401.8 (TXD)
- net LoRa_TRX: now also U401.7 (RXD)
- net RF_switch1: now also C403.1, Switch401.6 (V2)
- net RF_switch2: now also C404.1, Switch401.4 (V1)
- net VDD: now also C406.1, C407.1, U401.10 (VDD)
- new net: C402.2, D402.2 (A2), J402.1 (In)
- new net: C401.1, Switch401.1 (J3)
- new net: C402.1, Switch401.3 (J2)
- new net: C405.2, Switch401.5 (J1)
- new net: C401.2, D401.2 (A2), J401.1 (In)
- new net: C405.1, U401.21 (ANT)
