File: hardware/modules/LoRa2026/ESP32Core.kicad_sch (KiCad schematic)
At the start: 22 parts, among them SW1 RESET_sw, U1 TPS3820, U2 SN65HVD230, U3 ESP32-S3-WROOM-1

Commit message: LoRa2026修正ver2
Parts:
- added SW702: RESET, WOBCLibrary:TVAF06-A020B-R, symbol Switch:SW_Push
- U701: renamed from U1; footprint PCM_Package_TO_SOT_SMD_AKL:SOT-23-5 -> Package_TO_SOT_SMD:SOT-23-5
- renumbered C1 to C701, C2 to C702, C3 to C703, C4 to C704, D1 to D701, D2 to D702, D3 to D703, D4 to D704, D5 to D705, D6 to D706, R1 to R701, R2 to R702, R3 to R703, R4 to R704, R5 to R705, R6 to R706, R7 to R707, SW1 to SW701, U2 to U702, U3 to U703, USB1 to USB701
Connections:
- net GND: now also SW702.2
- net at U703.27 (GPIO0/BOOT): now also SW702.1
- no-connect marks 9 -> 8
Other:
- moved on the sheet: C703, C704, D705, D706, R704, R705, R706, R707, U703

Commit message: LoRa2026修正ver3
Parts:
- USB701: LCSC C2856766 -> C720625
Changed lines of the file:
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@@
 			)
 		)
-		(property "LCSC" "C2856766"
+		(property "LCSC" "C720625"
 			(at 28.575 41.91 0)
 			(effects
